File: Robocup_PCB.kicad_pcb (KiCad board)
At the start: 2 copper layers, 209.8 x 196.2 mm, 55 parts, among them J1 M1_ENOUT, J2 M1_IN, J3 M2_ENOUT, J4 M2_IN, J5 M3_ENOUT, J6 M3_IN, J7 Arduino_Mega_Header, J8 XT60-M, Q1 IRF9540N, Q2 IRFR120ZTRPBF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

Commit message: BOM list generated
Parts:
- removed Q2: IRFR120ZTRPBF, 3rd party libs:DPAK229P990X239-3N
- added C13: 10n, Capacitor_SMD:C_0603_1608Metric_Pad1.05x0.95mm_HandSolder, F.Cu at (214.0, 186.7)
- added D3: RED, LED_SMD:LED_0805_2012Metric_Pad1.15x1.40mm_HandSolder, F.Cu at (286.5, 146.5)
- added D4: BLUE, LED_SMD:LED_0805_2012Metric_Pad1.15x1.40mm_HandSolder, F.Cu at (275.7, 158.7)
- added R15: 680R, Resistor_SMD:R_1206_3216Metric_Pad1.42x1.75mm_HandSolder, F.Cu at (276.3, 155.6)
- added R16: 180R, Resistor_SMD:R_1206_3216Metric_Pad1.42x1.75mm_HandSolder, F.Cu at (202.9, 187.0)
- added SW2: SS ESP101, Connector_PinSocket_2.54mm:PinSocket_1x03_P2.54mm_Vertical, F.Cu at (298.2, 109.8)
- added SW3: SS ESP101, Connector_PinSocket_2.54mm:PinSocket_1x03_P2.54mm_Vertical, F.Cu at (280.4, 125.4)
- added U5: TB6612FNG_MOD, Robocup_PCB:U_TB6612FNG_MOD, F.Cu at (269.9, 120.0)
- R13: footprint Resistor_SMD:R_1206_3216Metric_Pad1.42x1.75mm_HandSolder -> Resistor_SMD:R_0805_2012Metric_Pad1.15x1.40mm_HandSolder
- R14: value 140R -> 680R
- moved R1 202.7 mm to (294.4, 136.9)
- moved R2 201.2 mm to (299.0, 132.5)
- moved R6 176.4 mm to (257.3, 172.9)
- moved R11 170.3 mm to (240.5, 188.2)
- moved R3 167.9 mm to (267.5, 168.2)
- moved R7 161.0 mm to (299.0, 125.9)
- moved IR6 143.5 mm to (291.7, 123.8)
- moved R9 117.4 mm to (299.0, 129.2)
- moved IR9 116.8 mm to (282.5, 139.6)
- moved R4 113.7 mm to (208.8, 187.0)
- moved R13 111.3 mm to (281.6, 153.0)
- moved IR4 108.1 mm to (250.0, 172.0)
- moved IR2 108.1 mm to (248.9, 162.9)
- moved IR1 108.0 mm to (240.1, 162.9)
- moved R8 107.1 mm to (234.5, 188.2)
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Connections:
- D2 pad 1: Net-(D2-Pad1) -> GND
- J7 pad 54: Net-(J7-Pad54) -> M3_AIN2
- J7 pad 55: Net-(J7-Pad55) -> M3_AIN1
- J7 pad 56: Net-(J7-Pad56) -> M2_BIN2
- J7 pad 57: Net-(J7-Pad57) -> M2_BIN1
- J7 pad 58: Net-(J7-Pad58) -> M1_AIN2
- J7 pad 59: Net-(J7-Pad59) -> M1_AIN1
- J7 pad 71: M1_AIN1 -> Net-(J7-Pad71)
- J7 pad 72: M1_AIN2 -> Net-(J7-Pad72)
- J7 pad 74: M2_BIN1 -> Net-(J7-Pad74)
- J7 pad 75: M2_BIN2 -> Net-(J7-Pad75)
- J7 pad 77: M3_AIN1 -> Net-(J7-Pad77)
- J7 pad 78: M3_AIN2 -> Net-(J7-Pad78)
- J7 pad 79: M2_PWMB -> M3_PWMA
- Q1 pad 3: Net-(D1-Pad1) -> Net-(Q1-Pad3)
- R14 pad 1: Net-(D2-Pad2) -> +12V
- R14 pad 2: Net-(R14-Pad2) -> Net-(D2-Pad2)
- SW1 pad 1: +5V -> Net-(C13-Pad1)
- SW1 pad 2: Net-(R14-Pad2) -> GND
- U1 pad 11: M2_B -> Net-(U1-Pad11)
- U1 pad 12: M2_A -> Net-(U1-Pad12)
- U1 pad 5: M2_BIN1 -> Net-(U1-Pad5)
- U1 pad 6: M2_BIN2 -> Net-(U1-Pad6)
- U1 pad 7: M2_PWMB -> Net-(U1-Pad7)
- U2 pad 1: M3_PWMA -> Net-(U2-Pad1)
- U2 pad 11: Net-(U2-Pad11) -> M2_B
- U2 pad 12: Net-(U2-Pad12) -> M2_A
- U2 pad 13: M3_B -> Net-(U2-Pad13)
- U2 pad 14: M3_A -> Net-(U2-Pad14)
- U2 pad 2: M3_AIN2 -> Net-(U2-Pad2)
- U2 pad 3: M3_AIN1 -> Net-(U2-Pad3)
- U2 pad 5: Net-(U2-Pad5) -> M2_BIN1
- U2 pad 6: Net-(U2-Pad6) -> M2_BIN2
- U2 pad 7: Net-(U2-Pad7) -> M2_PWMB
- U3 pad 2: Net-(D1-Pad1) -> Net-(SW2-Pad2)
- U4 pad 2: Net-(Q2-Pad3) -> Net-(Q1-Pad3)
- U4 pad 3: Net-(U4-Pad3) -> Net-(C13-Pad1)

Commit message: Finished PCB, Generated Gerbers
Parts:
- removed J5: M3_ENOUT, Connector_PinSocket_2.54mm:PinSocket_1x02_P2.54mm_Vertical
- removed J6: M3_IN, Connector_PinSocket_2.54mm:PinSocket_1x06_P2.54mm_Vertical
- removed J7: Arduino_Mega_Header, w_conn_misc:arduino_mega_header
- removed SW1, SW2, SW3: SS ESP101, Connector_PinSocket_2.54mm:PinSocket_1x03_P2.54mm_Vertical
- added SW_ARD: SS ESP101, Connector_PinSocket_2.54mm:PinSocket_1x03_P2.54mm_Vertical, F.Cu at (209.6, 87.0)
- added SW_M: SS ESP101, Connector_PinSocket_2.54mm:PinSocket_1x03_P2.54mm_Vertical, F.Cu at (272.4, 81.9)
- added SW_P: SS ESP101, Connector_PinSocket_2.54mm:PinSocket_1x03_P2.54mm_Vertical, F.Cu at (264.2, 106.7)
- C13: footprint Capacitor_SMD:C_0603_1608Metric_Pad1.05x0.95mm_HandSolder -> Capacitor_SMD:C_1206_3216Metric_Pad1.42x1.75mm_HandSolder
- J1: value M1_ENOUT -> M1_IN; footprint Connector_PinSocket_2.54mm:PinSocket_1x02_P2.54mm_Vertical -> Connector_PinSocket_2.54mm:PinSocket_1x06_P2.54mm_Vertical
- J2: value M1_IN -> M2_IN
- J3: value M2_ENOUT -> M3_IN; footprint Connector_PinSocket_2.54mm:PinSocket_1x02_P2.54mm_Vertical -> Connector_PinSocket_2.54mm:PinSocket_1x06_P2.54mm_Vertical
- J4: value M2_IN -> Arduino_Mega_Header; footprint Connector_PinSocket_2.54mm:PinSocket_1x06_P2.54mm_Vertical -> w_conn_misc:arduino_mega_header
- Q1: footprint Package_TO_SOT_THT:TO-220-3_Vertical -> Package_TO_SOT_SMD:TO-263-2
- R13: footprint Resistor_SMD:R_0805_2012Metric_Pad1.15x1.40mm_HandSolder -> Resistor_SMD:R_1206_3216Metric_Pad1.42x1.75mm_HandSolder
- moved IR10 176.1 mm to (115.6, 127.0), turned to 270 degrees
- moved R9 173.0 mm to (132.1, 174.6), turned to 30 degrees
- moved IR12 161.5 mm to (154.2, 48.0), turned to 210 degrees
- moved R11 160.6 mm to (133.3, 68.6), turned to 60 degrees
- moved IR9 157.9 mm to (129.5, 179.1), turned to 300 degrees
- moved R12 155.8 mm to (158.8, 50.2), turned to 300 degrees
- moved IR11 152.4 mm to (130.8, 76.2), turned to 240 degrees
- moved C12 134.3 mm to (160.0, 55.2), turned to 30 degrees
- moved R7 131.4 mm to (214.6, 226.7), turned to 90 degrees
- moved C2 130.0 mm to (278.1, 58.4), turned to 330 degrees
- moved C13 125.6 mm to (273.7, 76.2)
- moved C11 125.2 mm to (136.5, 70.5), turned to 60 degrees
- moved R4 119.4 mm to (313.5, 129.5), turned to 180 degrees
- moved IR8 119.1 mm to (166.9, 216.2), turned to 330 degrees
- moved IR2 118.1 mm to (281.9, 49.5), turned to 150 degrees
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Connections:
- J1 pad 1: Net-(J1-Pad1) -> M1_A
- J1 pad 2: Net-(J1-Pad2) -> M1_B
- J2 pad 1: M1_A -> M2_A
- J2 pad 2: M1_B -> M2_B
- J2 pad 5: Net-(J1-Pad2) -> M2_ENA
- J2 pad 6: Net-(J1-Pad1) -> M2_ENB
- J3 pad 1: Net-(J3-Pad1) -> M3_A
- J3 pad 2: Net-(J3-Pad2) -> M3_B
- J4 pad 1: M2_A -> (no net)
- J4 pad 2: M2_B -> Net-(J4-Pad2)
- J4 pad 3: GND -> Net-(J4-Pad3)
- J4 pad 4: +5V -> +3V3
- J4 pad 5: Net-(J3-Pad2) -> +5V
- J4 pad 6: Net-(J3-Pad1) -> GND
- U3 pad 4: (no net) -> +5V
Routing:
- net +3V3: track 0.00 -> 674.1 mm, vias 0 -> 4
- net A1: track 0.00 -> 266.1 mm, vias 0 -> 6
- net A2: track 0.00 -> 246.9 mm, vias 0 -> 4
- net +5V: track 0.00 -> 246.0 mm, vias 0 -> 4
- net A10: track 0.00 -> 222.1 mm, vias 0 -> 2
- net A11: track 0.00 -> 202.1 mm, vias 0 -> 1
- net A0: track 0.00 -> 200.5 mm, vias 0 -> 2
- net A3: track 0.00 -> 156.5 mm, vias 0 -> 3
- net A9: track 0.00 -> 151.8 mm
- net M3_AIN1: track 0.00 -> 146.5 mm, vias 0 -> 2
- net M3_AIN2: track 0.00 -> 140.3 mm
- net +12V: track 0.00 -> 136.5 mm
- net A8: track 0.00 -> 118.2 mm
- net Net-(Q1-Pad3): track 0.00 -> 117.6 mm, vias 0 -> 1
- net M2_BIN2: track 0.00 -> 92.2 mm, vias 0 -> 1
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- added copper zone on B.Cu, net GND
- added copper zone on F.Cu, net GND
Other:
- net class Default: clearance 0.2 -> 0.5; trace_width 0.25 -> 0.254
- rule pad_to_mask_clearance: 0.051 -> 0.05
- rule solder_mask_min_width: 0.25 -> 0.2
- rule trace_clearance: 0.2 -> 0.5
- rule trace_min: 0.2 -> 0.254
- rule via_min_drill: 0.3 -> 0.305
- rule via_min_size: 0.4 -> 0.61
- board text added: "Off"
- board text added: "On"
- board text added: "Robocup PCB v1"
