File: Robocup_PCB.sch (KiCad schematic (older format))
At the start: 59 parts, among them J1 M1_IN, J2 M2_IN, J3 M3_IN, J4 Arduino_Mega_Header, J8 XT60-M, Q1 IRF9540N, SW1 SS ESP101, SW2 SS ESP101, SW3 SS ESP101, U1 TB6612FNG_MOD, U2 TB6612FNG_MOD, U3 5V_D24V5F5, U4 12V_S18V20F12, U5 TB6612FNG_MOD

Commit message: 5V regulator done
Parts:
- removed U3: 5V_D24V5F5, symbol Robocup_PCB:5V_D24V5F5
- added C?: 22uF, symbol Device:C
- added C?: 10uF, symbol Device:C
- added L?: 2.2uH, symbol Device:L
- added R? (x2): 100k, symbol Device:R
- added R?: 12k, symbol Device:R
- added R?: 63k, symbol Device:R
- added U?: TI_TPS62170DSGR, symbol Robocup_PCB:TI_TPS62170DSGR
Connections:
- net labels added: VDC
- wire segments 223 -> 254
- no-connect marks 73 -> 77
Other:
- moved on the sheet: C13, D1, D2, D3, D4, J1, J2, J3, J4, J8, Q1, R13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

Commit message: Started Light PCB
Parts:
- gave numbers to parts that had none: 8
Changed lines of the file:
@@
 NoConn ~ 1400 5850
 $Comp
-L power:VDC #PWR?
+L power:VDC #PWR017
 U 1 1 60634485
 P 8900 2150
-F 0 "#PWR?" H 8900 2050 50  0001 C CNN
+F 0 "#PWR017" H 8900 2050 50  0001 C CNN
 F 1 "VDC" H 8915 2323 50  0000 C CNN
 F 2 "" H 8900 2150 50  0001 C CNN
@@
 $EndComp
 $Comp
-L power:GND #PWR?
+L power:GND #PWR020
 U 1 1 60A20084
 P 10750 3100
-F 0 "#PWR?" H 10750 2850 50  0001 C CNN
+F 0 "#PWR020" H 10750 2850 50  0001 C CNN
 F 1 "GND" V 10755 2972 50  0000 R CNN
 F 2 "" H 10750 3100 50  0001 C CNN
@@
 $EndComp
 $Comp
-L power:VDC #PWR?
+L power:VDC #PWR01
 U 1 1 60B8520C
 P 7150 5400
-F 0 "#PWR?" H 7150 5300 50  0001 C CNN
+F 0 "#PWR01" H 7150 5300 50  0001 C CNN
 F 1 "VDC" H 7165 5573 50  0000 C CNN
 F 2 "" H 7150 5400 50  0001 C CNN
@@
 	8350 5700 8500 5700
 $Comp
-L power:GND #PWR?
+L power:GND #PWR016
 U 1 1 60BA077F
 P 8350 5750
-F 0 "#PWR?" H 8350 5500 50  0001 C CNN
+F 0 "#PWR016" H 8350 5500 50  0001 C CNN
 F 1 "GND" V 8355 5622 50  0000 R CNN
 F 2 "" H 8350 5750 50  0001 C CNN
@@
 Connection ~ 8350 5700
 $Comp
-L Device:L L?
+L Device:L L1
 U 1 1 60BE3626
 P 9350 5400
-F 0 "L?" V 9540 5400 50  0000 C CNN
+F 0 "L1" V 9540 5400 50  0000 C CNN
 F 1 "2.2uH" V 9449 5400 50  0000 C CNN
 F 2 "" H 9350 5400 50  0001 C CNN
@@
 	9200 5400 9100 5400
 $Comp
-L Device:R R?
+L Device:R R18
 U 1 1 60BF1E65
 P 9350 5600
-F 0 "R?" H 9420 5646 50  0000 L CNN
+F 0 "R18" H 9420 5646 50  0000 L CNN
 F 1 "100k" H 9420 5555 50  0000 L CNN
 F 2 "" V 9280 5600 50  0001 C CNN
@@
 $EndComp
 $Comp
-L Device:R R?
+L Device:R R20
 U 1 1 60BF30CA
 P 9800 6000
-F 0 "R?" H 9730 5954 50  0000 R CNN
+F 0 "R20" H 9730 5954 50  0000 R CNN
 F 1 "12k" H 9730 6045 50  0000 R CNN
 F 2 "" V 9730 6000 50  0001 C CNN
@@
 	9600 5500 9600 5400
 $Comp
-L power:GND #PWR?
+L power:GND #PWR018
 U 1 1 60CA7826
 P 9800 6200
-F 0 "#PWR?" H 9800 5950 50  0001 C CNN
+F 0 "#PWR018" H 9800 5950 50  0001 C CNN
 F 1 "GND" V 9805 6072 50  0000 R CNN
 F 2 "" H 9800 6200 50  0001 C CNN
@@
 $EndComp
 $Comp
-L Device:C C?
+L Device:C C15
 U 1 1 60CD59FE
 P 10100 5600
-F 0 "C?" H 10215 5646 50  0000 L CNN
+F 0 "C15" H 10215 5646 50  0000 L CNN
 F 1 "22uF" H 10215 5555 50  0000 L CNN
 F 2 "" H 10138 5450 50  0001 C CNN
@@
 Connection ~ 7400 5400
 $Comp
-L power:GND #PWR?
+L power:GND #PWR02
 U 1 1 60D05CF1
 P 7400 6150
-F 0 "#PWR?" H 7400 5900 50  0001 C CNN
+F 0 "#PWR02" H 7400 5900 50  0001 C CNN
 F 1 "GND" V 7405 6022 50  0000 R CNN
 F 2 "" H 7400 6150 50  0001 C CNN
@@
 	7400 6150 7400 5900
 $Comp
-L power:+5V #PWR?
+L power:+5V #PWR021
 U 1 1 60D53F9F
 P 10850 5400
-F 0 "#PWR?" H 10850 5250 50  0001 C CNN
+F 0 "#PWR021" H 10850 5250 50  0001 C CNN
 F 1 "+5V" V 10865 5528 50  0000 L CNN
 F 2 "" H 10850 5400 50  0001 C CNN
@@
 	9800 6150 9800 6200
 $Comp
-L power:GND #PWR?
+L power:GND #PWR019
 U 1 1 60D561CF
 P 10100 6200
-F 0 "#PWR?" H 10100 5950 50  0001 C CNN
+F 0 "#PWR019" H 10100 5950 50  0001 C CNN
 F 1 "GND" V 10105 6072 50  0000 R CNN
 F 2 "" H 10100 6200 50  0001 C CNN
@@
 	10100 5750 10100 6200
 $Comp
-L Device:R R?
+L Device:R R19
 U 1 1 60BF363B
 P 9800 5600
-F 0 "R?" H 9730 5554 50  0000 R CNN
+F 0 "R19" H 9730 5554 50  0000 R CNN
 F 1 "63k" H 9730 5645 50  0000 R CNN
 F 2 "" V 9730 5600 50  0001 C CNN
@@
 $EndComp
 $Comp
-L Device:C C?
+L Device:C C14
 U 1 1 60CF5B3B
 P 7400 5750
-F 0 "C?" H 7515 5796 50  0000 L CNN
+F 0 "C14" H 7515 5796 50  0000 L CNN
 F 1 "10uF" H 7515 5705 50  0000 L CNN
 F 2 "" H 7438 5600 50  0001 C CNN
@@
 	8300 5550 8300 5500
 $Comp
-L power:GND #PWR?
+L power:GND #PWR015
 U 1 1 60DC24F8
 P 7750 6150
-F 0 "#PWR?" H 7750 5900 50  0001 C CNN
+F 0 "#PWR015" H 7750 5900 50  0001 C CNN
 F 1 "GND" V 7755 6022 50  0000 R CNN
 F 2 "" H 7750 6150 50  0001 C CNN
@@
 $EndComp
 $Comp
-L Device:R R?
+L Device:R R17
 U 1 1 60DC31B4
 P 7750 5950
-F 0 "R?" H 7680 5904 50  0000 R CNN
+F 0 "R17" H 7680 5904 50  0000 R CNN
 F 1 "100k" H 7680 5995 50  0000 R CNN
 F 2 "" V 7680 5950 50  0001 C CNN
@@
 	7750 5650 7850 5650
 $Comp
-L Robocup_PCB:TI_TPS62170DSGR U?
+L Robocup_PCB:TI_TPS62170DSGR U3
 U 1 1 60DF4FCF
 P 8800 5800
-F 0 "U?" H 8800 6425 50  0000 C CNN
+F 0 "U3" H 8800 6425 50  0000 C CNN
 F 1 "TI_TPS62170DSGR" H 8800 6334 50  0000 C CNN
 F 2 "" H 8800 5800 50  0001 C CNN

Commit message: Started MUX
Parts:
- added U?: AD_ADG732, symbol Robocup_PCB:AD_ADG732
- C1, C10, C11, C12, C2, C3, C4, C5, C6, C7, C8, C9: value 0.1uF -> 4.7u
- R1, R11, R12, R2, R3, R4, R5, R6, R7, R8, R9: value 6k2 -> 2k2
- renumbered C15 to C?, C14 to C?, L1 to L?, R18 to R?, R20 to R?, R19 to R?, R17 to R?, U3 to U?
Connections:
- net +5V: now also U?.13 (VDD), U?.14 (VDD)
- net GND: now also U?.23 (GND)
- no-connect marks 77 -> 82
Other:
- moved on the sheet: C1, C10, C11, C12, C13, C2, C3, C4, C5, C6, C7, C8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

Commit message: Finished MUX
Parts:
- removed C?: 22uF, symbol Device:C
- removed C?: 10uF, symbol Device:C
- removed D4: BLUE, LED_SMD:LED_0805_2012Metric_Pad1.15x1.40mm_HandSolder, symbol Device:LED
- removed L?: 2.2uH, symbol Device:L
- removed R16: 180R, Resistor_SMD:R_1206_3216Metric_Pad1.42x1.75mm_HandSolder, symbol Device:R
- removed R? (x2): 100k, symbol Device:R
- removed R?: 12k, symbol Device:R
- removed R?: 63k, symbol Device:R
- removed SW2: SS ESP101, Connector_PinSocket_2.54mm:PinSocket_1x03_P2.54mm_Vertical, symbol Switch:SW_SPDT
- removed U?: TI_TPS62170DSGR, symbol Robocup_PCB:TI_TPS62170DSGR
- added C?: 1u, symbol Device:C
- added C?: 0.1u, symbol Device:C
- added C? (x2): 10u, symbol Device:C
- added J?: Conn_02x13_Odd_Even, symbol Connector_Generic:Conn_02x13_Odd_Even
- added U?: NCP1117-5.0_TO252, Package_TO_SOT_SMD:TO-252-2, symbol Regulator_Linear:NCP1117-5.0_TO252
Connections:
- net +5V: now also C?.1, C?.2, C?.2, J?.26 (Pin_26), U?.2 (VO)
- net GND: now also U?.24 (Vss), C?.1, C?.1, C?.2, C?.2, J?.25 (Pin_25), U?.1 (GND)
- net A12: now reaches J4.21 (DAC0/CANRX1)
- net A12: now also U?.43 (D)
- net D36: now reaches J4.34 (PIN36)
- net D36: now also U?.22 (~EN)
- net D34: now reaches J4.35 (PIN34)
- net D34: now also U?.21 (~WR)
- net D32: now reaches J4.36 (PIN32)
- net D32: now also U?.20 (~CS)
- net D30: now reaches J4.37 (PIN30)
- net D30: now also U?.19 (A4)
- net D28: now reaches J4.38 (PIN28)
- net D28: now also U?.18 (A3)
- net D26: now reaches J4.39 (PIN26)
- net D26: now also U?.17 (A2)
- net D24: now reaches J4.40 (PIN24)
- net D24: now also U?.16 (A1)
- net D22: now reaches J4.41 (PIN22)
- net D22: now also U?.15 (A0)
- net S12: now reaches U?.1 (S12)
- net S12: now also J?.12 (Pin_12)
- net S3: now reaches U?.10 (S3)
- net S3: now also J?.3 (Pin_3)
- net S2: now reaches U?.11 (S2)
- net S2: now also J?.2 (Pin_2)
- net S1: now reaches U?.12 (S1)
- net S1: now also J?.1 (Pin_1)
- net S11: now reaches U?.2 (S11)
- net S11: now also J?.11 (Pin_11)
- net S17: now reaches U?.25 (S17)
- net S17: now also J?.17 (Pin_17)
- net S18: now reaches U?.26 (S18)
- net S18: now also J?.18 (Pin_18)
- net S19: now reaches U?.27 (S19)
- net S19: now also J?.19 (Pin_19)
- net S20: now reaches U?.28 (S20)
- net S20: now also J?.20 (Pin_20)
- net S21: now reaches U?.29 (S21)
- net S21: now also J?.21 (Pin_21)
- net S10: now reaches U?.3 (S10)
- net S10: now also J?.10 (Pin_10)
- net S22: now reaches U?.30 (S22)
- net S22: now also J?.22 (Pin_22)
- net S23: now reaches U?.31 (S23)
- net S23: now also J?.23 (Pin_23)
- net S24: now reaches U?.32 (S24)
- net S24: now also J?.24 (Pin_24)
- net S9: now reaches U?.4 (S9)
- net S9: now also J?.9 (Pin_9)
- net S16: now reaches U?.45 (S16)
- net S16: now also J?.16 (Pin_16)
- net S15: now reaches U?.46 (S15)
- net S15: now also J?.15 (Pin_15)
- net S14: now reaches U?.47 (S14)
- net S14: now also J?.14 (Pin_14)
- net S13: now reaches U?.48 (S13)
- net S13: now also J?.13 (Pin_13)
- net S8: now reaches U?.5 (S8)
- net S8: now also J?.8 (Pin_8)
- net S7: now reaches U?.6 (S7)
- net S7: now also J?.7 (Pin_7)
- net S6: now reaches U?.7 (S6)
- net S6: now also J?.6 (Pin_6)
- net S5: now reaches U?.8 (S5)
- net S5: now also J?.5 (Pin_5)
- net S4: now reaches U?.9 (S4)
- net S4: now also J?.4 (Pin_4)
- net VDC renamed +VDC
- net +VDC: now also C?.1, U?.3 (VI)
- no-connect marks 82 -> 79
Other:
- moved on the sheet: C13, D1, D2, D3, J8, Q1, R13, R14, R15, SW1, SW3, U4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

Commit message: Finished Motor Drivers
Parts:
- removed U1, U2, U5: TB6612FNG_MOD, Robocup_PCB:U_TB6612FNG_MOD, symbol Robocup_PCB:TB6612FNG_MOD
- gave numbers to parts that had none: 7
Connections:
- net +5V: no longer J1.4 (Pin_4), J2.4 (Pin_4), J3.4 (Pin_4)
- net GND: no longer J1.3 (Pin_3), J2.3 (Pin_3), J3.3 (Pin_3)
- net M1_ENA: no longer names the net of J1.5 (Pin_5)
- net M1_ENB: no longer names the net of J1.6 (Pin_6)
- net M2_ENA: no longer names the net of J2.5 (Pin_5)
- net M2_ENB: no longer names the net of J2.6 (Pin_6)
- net M3_ENA: no longer names the net of J3.5 (Pin_5)
- net M3_ENB: no longer names the net of J3.6 (Pin_6)
- no-connect marks 79 -> 66

Commit message: Finished Light Ring Schematic
Other:
- moved on the sheet: J5
Changed lines of the file:
@@
 L Connector_Generic:Conn_02x13_Odd_Even J5
 U 1 1 607C19C7
-P 4100 8200
-F 0 "J5" H 4150 9017 50  0000 C CNN
-F 1 "Conn_02x13_Odd_Even" H 4150 8926 50  0000 C CNN
-F 2 "" H 4100 8200 50  0001 C CNN
-F 3 "~" H 4100 8200 50  0001 C CNN
-	1    4100 8200
+P 3850 7800
+F 0 "J5" H 3900 8617 50  0000 C CNN
+F 1 "Conn_02x13_Odd_Even" H 3900 8526 50  0000 C CNN
+F 2 "" H 3850 7800 50  0001 C CNN
+F 3 "~" H 3850 7800 50  0001 C CNN
+	1    3850 7800
 	1    0    0    -1
 $EndComp
-Text GLabel 3800 7600 0    50   Output ~ 0
+Text GLabel 3550 7200 0    50   Output ~ 0
 S1
-Text GLabel 3800 7700 0    50   Output ~ 0
+Text GLabel 3550 7300 0    50   Output ~ 0
 S3
-Text GLabel 3800 7800 0    50   Output ~ 0
+Text GLabel 3550 7400 0    50   Output ~ 0
 S5
-Text GLabel 3800 7900 0    50   Output ~ 0
+Text GLabel 3550 7500 0    50   Output ~ 0
 S7
-Text GLabel 3800 8000 0    50   Output ~ 0
+Text GLabel 3550 7600 0    50   Output ~ 0
 S9
-Text GLabel 3800 8100 0    50   Output ~ 0
+Text GLabel 3550 7700 0    50   Output ~ 0
 S11
-Text GLabel 3800 8200 0    50   Output ~ 0
+Text GLabel 3550 7800 0    50   Output ~ 0
 S13
-Text GLabel 3800 8300 0    50   Output ~ 0
+Text GLabel 3550 7900 0    50   Output ~ 0
 S15
-Text GLabel 3800 8400 0    50   Output ~ 0
+Text GLabel 3550 8000 0    50   Output ~ 0
 S17
-Text GLabel 3800 8500 0    50   Output ~ 0
+Text GLabel 3550 8100 0    50   Output ~ 0
 S19
-Text GLabel 3800 8600 0    50   Output ~ 0
+Text GLabel 3550 8200 0    50   Output ~ 0
 S21
-Text GLabel 3800 8700 0    50   Output ~ 0
+Text GLabel 3550 8300 0    50   Output ~ 0
 S23
-Text GLabel 4500 7600 2    50   Output ~ 0
+Text GLabel 4250 7200 2    50   Output ~ 0
 S2
-Text GLabel 4500 7700 2    50   Output ~ 0
+Text GLabel 4250 7300 2    50   Output ~ 0
 S4
-Text GLabel 4500 7800 2    50   Output ~ 0
+Text GLabel 4250 7400 2    50   Output ~ 0
 S6
-Text GLabel 4500 7900 2    50   Output ~ 0
+Text GLabel 4250 7500 2    50   Output ~ 0
 S8
-Text GLabel 4500 8000 2    50   Output ~ 0
+Text GLabel 4250 7600 2    50   Output ~ 0
 S10
-Text GLabel 4500 8100 2    50   Output ~ 0
+Text GLabel 4250 7700 2    50   Output ~ 0
 S12
-Text GLabel 4500 8500 2    50   Output ~ 0
+Text GLabel 4250 8100 2    50   Output ~ 0
 S20
-Text GLabel 4500 8600 2    50   Output ~ 0
+Text GLabel 4250 8200 2    50   Output ~ 0
 S22
-Text GLabel 4500 8700 2    50   Output ~ 0
+Text GLabel 4250 8300 2    50   Output ~ 0
 S24
 Wire Wire Line
-	3800 7600 3900 7600
+	3550 7200 3650 7200
 Wire Wire Line
-	3800 7700 3900 7700
+	3550 7300 3650 7300
 Wire Wire Line
-	3800 7800 3900 7800
+	3550 7400 3650 7400
 Wire Wire Line
-	3800 7900 3900 7900
+	3550 7500 3650 7500
 Wire Wire Line
-	3800 8000 3900 8000
+	3550 7600 3650 7600
 Wire Wire Line
-	3800 8100 3900 8100
+	3550 7700 3650 7700
 Wire Wire Line
-	3800 8200 3900 8200
+	3550 7800 3650 7800
 Wire Wire Line
-	3800 8300 3900 8300
+	3550 7900 3650 7900
 Wire Wire Line
-	3800 8400 3900 8400
+	3550 8000 3650 8000
 Wire Wire Line
-	3800 8500 3900 8500
+	3550 8100 3650 8100
 Wire Wire Line
-	3800 8600 3900 8600
+	3550 8200 3650 8200
 Wire Wire Line
-	3800 8700 3900 8700
+	3550 8300 3650 8300
 Wire Wire Line
-	4400 8700 4500 8700
+	4150 8300 4250 8300
 Wire Wire Line
-	4400 8600 4500 8600
+	4150 8200 4250 8200
 Wire Wire Line
-	4400 8500 4500 8500
+	4150 8100 4250 8100
 Wire Wire Line
-	4400 8400 4500 8400
+	4150 8000 4250 8000
 Wire Wire Line
-	4400 8300 4500 8300
+	4150 7900 4250 7900
 Wire Wire Line
-	4400 8200 4500 8200
+	4150 7800 4250 7800
 Wire Wire Line
-	4400 8100 4500 8100
+	4150 7700 4250 7700
 Wire Wire Line
-	4400 8000 4500 8000
+	4150 7600 4250 7600
 Wire Wire Line
-	4400 7900 4500 7900
+	4150 7500 4250 7500
 Wire Wire Line
-	4400 7800 4500 7800
+	4150 7400 4250 7400
 Wire Wire Line
-	4400 7700 4500 7700
+	4150 7300 4250 7300
 Wire Wire Line
-	4400 7600 4500 7600
+	4150 7200 4250 7200
 $Comp
 L power:GND #PWR0129
 U 1 1 609C9542
-P 3800 8850
-F 0 "#PWR0129" H 3800 8600 50  0001 C CNN
-F 1 "GND" V 3805 8722 50  0000 R CNN
-F 2 "" H 3800 8850 50  0001 C CNN
-F 3 "" H 3800 8850 50  0001 C CNN
-	1    3800 8850
+P 3550 8450
+F 0 "#PWR0129" H 3550 8200 50  0001 C CNN
+F 1 "GND" V 3555 8322 50  0000 R CNN
+F 2 "" H 3550 8450 50  0001 C CNN
+F 3 "" H 3550 8450 50  0001 C CNN
+	1    3550 8450
 	1    0    0    -1
 $EndComp
@@
 L power:+5V #PWR0130
 U 1 1 609CA8AB
-P 4500 8850
-F 0 "#PWR0130" H 4500 8700 50  0001 C CNN
-F 1 "+5V" V 4515 8978 50  0000 L CNN
-F 2 "" H 4500 8850 50  0001 C CNN
-F 3 "" H 4500 8850 50  0001 C CNN
-	1    4500 8850
+P 4250 8450
+F 0 "#PWR0130" H 4250 8300 50  0001 C CNN
+F 1 "+5V" V 4265 8578 50  0000 L CNN
+F 2 "" H 4250 8450 50  0001 C CNN
+F 3 "" H 4250 8450 50  0001 C CNN
+	1    4250 8450
 	-1   0    0    1
 $EndComp
 Wire Wire Line
-	4500 8850 4500 8800
+	4250 8450 4250 8400
 Wire Wire Line
-	4500 8800 4400 8800
+	4250 8400 4150 8400
 Wire Wire Line
-	3800 8850 3800 8800
+	3550 8450 3550 8400
 Wire Wire Line
-	3800 8800 3900 8800
+	3550 8400 3650 8400
 NoConn ~ 2900 7200
 NoConn ~ 2900 7300
@@
 Text GLabel 1450 6800 1    50   Input ~ 0
 S13
-Text GLabel 4500 8200 2    50   Output ~ 0
+Text GLabel 4250 7800 2    50   Output ~ 0
 S14
 Text GLabel 1550 6800 1    50   Input ~ 0
@@
 Text GLabel 1650 6800 1    50   Input ~ 0
 S15
-Text GLabel 4500 8300 2    50   Output ~ 0
+Text GLabel 4250 7900 2    50   Output ~ 0
 S16
 Text GLabel 1750 6800 1    50   Input ~ 0
@@
 Text GLabel 3000 8300 2    50   Input ~ 0
 S17
-Text GLabel 4500 8400 2    50   Output ~ 0
+Text GLabel 4250 8000 2    50   Output ~ 0
 S18
 Text GLabel 3000 8200 2    50   Input ~ 0

Commit message: Started light pcb
Connections:
- net +VDC: now also R13.2
- net GND: no longer R13.2
Changed lines of the file:
@@
 Wire Wire Line
 	13250 1450 13400 1450
-$Comp
-L power:GND #PWR0146
-U 1 1 603A3E0E
-P 12750 1450
-F 0 "#PWR0146" H 12750 1200 50  0001 C CNN
-F 1 "GND" V 12755 1322 50  0000 R CNN
-F 2 "" H 12750 1450 50  0001 C CNN
-F 3 "" H 12750 1450 50  0001 C CNN
-	1    12750 1450
-	1    0    0    -1
-$EndComp
 Wire Wire Line
 	12750 1450 12950 1450
@@
 	0    1    1    0
 $EndComp
+$Comp
+L power:+VDC #PWR?
+U 1 1 6081D8C4
+P 12750 1450
+F 0 "#PWR?" H 12750 1350 50  0001 C CNN
+F 1 "+VDC" H 12750 1725 50  0000 C CNN
+F 2 "" H 12750 1450 50  0001 C CNN
+F 3 "" H 12750 1450 50  0001 C CNN
+	1    12750 1450
+	1    0    0    -1
+$EndComp
 $EndSCHEMATC
