File: OLD/Robocup_PCB.kicad_pcb (KiCad board)
At the start: 2 copper layers, 209.8 x 196.2 mm, 59 parts, among them J1 M1_IN, J2 M2_IN, J3 M3_IN, J4 Arduino_Mega_Header, J8 XT60-M, Q1 IRF9540N, U1 TB6612FNG_MOD, U2 TB6612FNG_MOD, U3 5V_D24V5F5, U4 12V_S18V20F12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

Commit message: old stuff
Parts:
- moved C12 24.8 mm to (174.0, 75.7), turned to 180 degrees
- moved R12 24.1 mm to (172.5, 70.0), turned to 270 degrees
- moved C1 21.2 mm to (238.3, 73.8)
- moved R1 19.6 mm to (238.3, 70.0), turned to 0 degrees
- moved R7 18.3 mm to (232.9, 226.7)
- moved C7 18.3 mm to (236.1, 226.7)
- moved C8 15.8 mm to (185.9, 206.1)
- moved R8 15.8 mm to (182.8, 209.3)
- moved R2 15.5 mm to (271.9, 66.4), turned to 270 degrees
- moved C2 13.5 mm to (273.4, 71.1), turned to 180 degrees
- moved C10 13.2 mm to (137.7, 125.7)
- moved R10 13.2 mm to (133.2, 124.5)
- moved C9 12.2 mm to (148.7, 173.4)
- moved R9 12.2 mm to (144.3, 174.6)
- moved R6 10.5 mm to (254.0, 215.3)
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Routing:
- net Net-(IR12-Pad1): track 4.04 -> 31.3 mm
- net A11: track 202.1 -> 178.6 mm
- net A0: track 200.5 -> 222.6 mm
- net A6: track 63.0 -> 44.7 mm
- net Net-(IR7-Pad1): track 2.81 -> 19.5 mm
- net A7: track 74.2 -> 57.8 mm
- net A1: track 266.1 -> 249.8 mm
- net Net-(IR2-Pad1): track 4.33 -> 20.4 mm
- net Net-(IR8-Pad1): track 4.66 -> 20.0 mm
- net Net-(IR10-Pad1): track 4.08 -> 17.3 mm
- net Net-(IR1-Pad1): track 4.72 -> 17.1 mm
- net A8: track 118.2 -> 106.0 mm
- net Net-(IR9-Pad1): track 4.35 -> 16.5 mm
- net A10: track 222.1 -> 211.3 mm
- net Net-(IR11-Pad1): track 4.19 -> 14.9 mm
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