File: Light_Ring_PCB/Light_Ring_PCB.sch (KiCad schematic (older format))
At the start: 121 parts, among them J1 Conn_02x13_Odd_Even, Q1 Q_Photo_NPN, Q10 Q_Photo_NPN, Q11 Q_Photo_NPN, Q12 Q_Photo_NPN, Q13 Q_Photo_NPN, Q14 Q_Photo_NPN, Q15 Q_Photo_NPN, Q16 Q_Photo_NPN, Q17 Q_Photo_NPN, Q18 Q_Photo_NPN, Q19 Q_Photo_NPN, Q2 Q_Photo_NPN, Q20 Q_Photo_NPN, Q21 Q_Photo_NPN, Q22 Q_Photo_NPN, Q23 Q_Photo_NPN, Q24 Q_Photo_NPN, Q3 Q_Photo_NPN, Q4 Q_Photo_NPN, Q5 Q_Photo_NPN, Q6 Q_Photo_NPN, Q7 Q_Photo_NPN, Q8 Q_Photo_NPN, Q9 Q_Photo_NPN

Commit message: Finished Light Ring Schematic
Parts:
- removed J1: Conn_02x13_Odd_Even, symbol Connector_Generic:Conn_02x13_Odd_Even
- added J?: Conn_02x14_Odd_Even, symbol Connector_Generic:Conn_02x14_Odd_Even
- added Q?: 2N7000, Package_TO_SOT_THT:TO-92_Inline, symbol Transistor_FET:2N7000
- added R?: 100k, symbol Device:R
Connections:
- net labels added: EN
- wire segments 340 -> 346
- no-connect marks 0 -> 1
Other:
- moved on the sheet: C17, C18, C19, C20, C21, C22, C23, C24, D17, D18, D19, D20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

Commit message: Started light pcb
Parts:
- D1, D10, D11, D12, D13, D14, D15, D16, D17, D18, D19, D2, D20, D21, D22, D23, D24, D3, D4, D5, D6, D7, D8, D9: footprint (none) -> Robocup_PCB:LED_C210341
- J1: renamed from J?; footprint (none) -> Connector_PinHeader_2.00mm:PinHeader_2x14_P2.00mm_Vertical
- Q25: renamed from Q?; footprint Package_TO_SOT_THT:TO-92_Inline -> Package_TO_SOT_SMD:SOT-223
- R49: renamed from R?; footprint (none) -> Resistor_SMD:R_0603_1608Metric_Pad1.05x0.95mm_HandSolder
Changed lines of the file:
@@
 F 0 "D1" V 1639 1482 50  0000 R CNN
 F 1 "LED" V 1548 1482 50  0000 R CNN
-F 2 "" H 1600 1600 50  0001 C CNN
+F 2 "Robocup_PCB:LED_C210341" H 1600 1600 50  0001 C CNN
 F 3 "~" H 1600 1600 50  0001 C CNN
 	1    1600 1600
@@
 F 0 "D5" V 2839 1482 50  0000 R CNN
 F 1 "LED" V 2748 1482 50  0000 R CNN
-F 2 "" H 2800 1600 50  0001 C CNN
+F 2 "Robocup_PCB:LED_C210341" H 2800 1600 50  0001 C CNN
 F 3 "~" H 2800 1600 50  0001 C CNN
 	1    2800 1600
@@
 F 0 "D9" V 3989 1432 50  0000 R CNN
 F 1 "LED" V 3898 1432 50  0000 R CNN
-F 2 "" H 3950 1550 50  0001 C CNN
+F 2 "Robocup_PCB:LED_C210341" H 3950 1550 50  0001 C CNN
 F 3 "~" H 3950 1550 50  0001 C CNN
 	1    3950 1550
@@
 F 0 "D13" V 5189 1432 50  0000 R CNN
 F 1 "LED" V 5098 1432 50  0000 R CNN
-F 2 "" H 5150 1550 50  0001 C CNN
+F 2 "Robocup_PCB:LED_C210341" H 5150 1550 50  0001 C CNN
 F 3 "~" H 5150 1550 50  0001 C CNN
 	1    5150 1550
@@
 F 0 "D2" V 1639 3132 50  0000 R CNN
 F 1 "LED" V 1548 3132 50  0000 R CNN
-F 2 "" H 1600 3250 50  0001 C CNN
+F 2 "Robocup_PCB:LED_C210341" H 1600 3250 50  0001 C CNN
 F 3 "~" H 1600 3250 50  0001 C CNN
 	1    1600 3250
@@
 F 0 "D6" V 2839 3132 50  0000 R CNN
 F 1 "LED" V 2748 3132 50  0000 R CNN
-F 2 "" H 2800 3250 50  0001 C CNN
+F 2 "Robocup_PCB:LED_C210341" H 2800 3250 50  0001 C CNN
 F 3 "~" H 2800 3250 50  0001 C CNN
 	1    2800 3250
@@
 F 0 "D10" V 3989 3082 50  0000 R CNN
 F 1 "LED" V 3898 3082 50  0000 R CNN
-F 2 "" H 3950 3200 50  0001 C CNN
+F 2 "Robocup_PCB:LED_C210341" H 3950 3200 50  0001 C CNN
 F 3 "~" H 3950 3200 50  0001 C CNN
 	1    3950 3200
@@
 F 0 "D14" V 5189 3082 50  0000 R CNN
 F 1 "LED" V 5098 3082 50  0000 R CNN
-F 2 "" H 5150 3200 50  0001 C CNN
+F 2 "Robocup_PCB:LED_C210341" H 5150 3200 50  0001 C CNN
 F 3 "~" H 5150 3200 50  0001 C CNN
 	1    5150 3200
@@
 F 0 "D3" V 1639 4782 50  0000 R CNN
 F 1 "LED" V 1548 4782 50  0000 R CNN
-F 2 "" H 1600 4900 50  0001 C CNN
+F 2 "Robocup_PCB:LED_C210341" H 1600 4900 50  0001 C CNN
 F 3 "~" H 1600 4900 50  0001 C CNN
 	1    1600 4900
@@
 F 0 "D7" V 2839 4782 50  0000 R CNN
 F 1 "LED" V 2748 4782 50  0000 R CNN
-F 2 "" H 2800 4900 50  0001 C CNN
+F 2 "Robocup_PCB:LED_C210341" H 2800 4900 50  0001 C CNN
 F 3 "~" H 2800 4900 50  0001 C CNN
 	1    2800 4900
@@
 F 0 "D11" V 3989 4732 50  0000 R CNN
 F 1 "LED" V 3898 4732 50  0000 R CNN
-F 2 "" H 3950 4850 50  0001 C CNN
+F 2 "Robocup_PCB:LED_C210341" H 3950 4850 50  0001 C CNN
 F 3 "~" H 3950 4850 50  0001 C CNN
 	1    3950 4850
@@
 F 0 "D15" V 5189 4732 50  0000 R CNN
 F 1 "LED" V 5098 4732 50  0000 R CNN
-F 2 "" H 5150 4850 50  0001 C CNN
+F 2 "Robocup_PCB:LED_C210341" H 5150 4850 50  0001 C CNN
 F 3 "~" H 5150 4850 50  0001 C CNN
 	1    5150 4850
@@
 F 0 "D4" V 1639 6432 50  0000 R CNN
 F 1 "LED" V 1548 6432 50  0000 R CNN
-F 2 "" H 1600 6550 50  0001 C CNN
+F 2 "Robocup_PCB:LED_C210341" H 1600 6550 50  0001 C CNN
 F 3 "~" H 1600 6550 50  0001 C CNN
 	1    1600 6550
@@
 F 0 "D8" V 2839 6432 50  0000 R CNN
 F 1 "LED" V 2748 6432 50  0000 R CNN
-F 2 "" H 2800 6550 50  0001 C CNN
+F 2 "Robocup_PCB:LED_C210341" H 2800 6550 50  0001 C CNN
 F 3 "~" H 2800 6550 50  0001 C CNN
 	1    2800 6550
@@
 F 0 "D12" V 3989 6382 50  0000 R CNN
 F 1 "LED" V 3898 6382 50  0000 R CNN
-F 2 "" H 3950 6500 50  0001 C CNN
+F 2 "Robocup_PCB:LED_C210341" H 3950 6500 50  0001 C CNN
 F 3 "~" H 3950 6500 50  0001 C CNN
 	1    3950 6500
@@
 F 0 "D16" V 5189 6382 50  0000 R CNN
 F 1 "LED" V 5098 6382 50  0000 R CNN
-F 2 "" H 5150 6500 50  0001 C CNN
+F 2 "Robocup_PCB:LED_C210341" H 5150 6500 50  0001 C CNN
 F 3 "~" H 5150 6500 50  0001 C CNN
 	1    5150 6500
@@
 F 0 "D17" V 6389 4082 50  0000 R CNN
 F 1 "LED" V 6298 4082 50  0000 R CNN
-F 2 "" H 6350 4200 50  0001 C CNN
+F 2 "Robocup_PCB:LED_C210341" H 6350 4200 50  0001 C CNN
 F 3 "~" H 6350 4200 50  0001 C CNN
 	1    6350 4200
@@
 Connection ~ 7150 3950
 $Comp
-L Device:LED D19
-U 1 1 60A1DCFB
-P 7550 4200
-F 0 "D19" V 7589 4082 50  0000 R CNN
-F 1 "LED" V 7498 4082 50  0000 R CNN
-F 2 "" H 7550 4200 50  0001 C CNN
-F 3 "~" H 7550 4200 50  0001 C CNN
-	1    7550 4200
-	0    -1   -1   0
-$EndComp
-$Comp
 L power:+5V #PWR077
 U 1 1 60A1DD01
@@
 F 0 "D21" V 8739 4032 50  0000 R CNN
 F 1 "LED" V 8648 4032 50  0000 R CNN
-F 2 "" H 8700 4150 50  0001 C CNN
+F 2 "Robocup_PCB:LED_C210341" H 8700 4150 50  0001 C CNN
 F 3 "~" H 8700 4150 50  0001 C CNN
 	1    8700 4150
@@
 F 0 "D23" V 9939 4032 50  0000 R CNN
 F 1 "LED" V 9848 4032 50  0000 R CNN
-F 2 "" H 9900 4150 50  0001 C CNN
+F 2 "Robocup_PCB:LED_C210341" H 9900 4150 50  0001 C CNN
 F 3 "~" H 9900 4150 50  0001 C CNN
 	1    9900 4150
@@
 F 0 "D18" V 6389 5732 50  0000 R CNN
 F 1 "LED" V 6298 5732 50  0000 R CNN
-F 2 "" H 6350 5850 50  0001 C CNN
+F 2 "Robocup_PCB:LED_C210341" H 6350 5850 50  0001 C CNN
 F 3 "~" H 6350 5850 50  0001 C CNN
 	1    6350 5850
@@
 F 0 "D20" V 7589 5732 50  0000 R CNN
 F 1 "LED" V 7498 5732 50  0000 R CNN
-F 2 "" H 7550 5850 50  0001 C CNN
+F 2 "Robocup_PCB:LED_C210341" H 7550 5850 50  0001 C CNN
 F 3 "~" H 7550 5850 50  0001 C CNN
 	1    7550 5850
@@
 F 0 "D22" V 8739 5682 50  0000 R CNN
 F 1 "LED" V 8648 5682 50  0000 R CNN
-F 2 "" H 8700 5800 50  0001 C CNN
+F 2 "Robocup_PCB:LED_C210341" H 8700 5800 50  0001 C CNN
 F 3 "~" H 8700 5800 50  0001 C CNN
 	1    8700 5800
@@
 F 0 "D24" V 9939 5682 50  0000 R CNN
 F 1 "LED" V 9848 5682 50  0000 R CNN
-F 2 "" H 9900 5800 50  0001 C CNN
+F 2 "Robocup_PCB:LED_C210341" H 9900 5800 50  0001 C CNN
 F 3 "~" H 9900 5800 50  0001 C CNN
 	1    9900 5800
@@
 	8650 700  8750 700
 $Comp
-L Connector_Generic:Conn_02x14_Odd_Even J?
+L Connector_Generic:Conn_02x14_Odd_Even J1
 U 1 1 60F66837
 P 8350 1300
-F 0 "J?" H 8400 2117 50  0000 C CNN
+F 0 "J1" H 8400 2117 50  0000 C CNN
 F 1 "Conn_02x14_Odd_Even" H 8400 2026 50  0000 C CNN
-F 2 "" H 8350 1300 50  0001 C CNN
+F 2 "Connector_PinHeader_2.00mm:PinHeader_2x14_P2.00mm_Vertical" H 8350 1300 50  0001 C CNN
 F 3 "~" H 8350 1300 50  0001 C CNN
 	1    8350 1300
@@
 EN
 $Comp
-L Transistor_FET:2N7000 Q?
+L Transistor_FET:2N7000 Q25
 U 1 1 61268F06
 P 7950 2300
-F 0 "Q?" H 8154 2346 50  0000 L CNN
+F 0 "Q25" H 8154 2346 50  0000 L CNN
 F 1 "2N7000" H 8154 2255 50  0000 L CNN
-F 2 "Package_TO_SOT_THT:TO-92_Inline" H 8150 2225 50  0001 L CIN
+F 2 "Package_TO_SOT_SMD:SOT-223" H 8150 2225 50  0001 L CIN
 F 3 "https://www.fairchildsemi.com/datasheets/2N/2N7000.pdf" H 7950 2300 50  0001 L CNN
 	1    7950 2300
@@
 	8050 2750 8050 2500
 $Comp
-L Device:R R?
+L Device:R R49
 U 1 1 6128CA16
 P 7600 2500
-F 0 "R?" H 7670 2546 50  0000 L CNN
+F 0 "R49" H 7670 2546 50  0000 L CNN
 F 1 "100k" H 7670 2455 50  0000 L CNN
-F 2 "" V 7530 2500 50  0001 C CNN
+F 2 "Resistor_SMD:R_0603_1608Metric_Pad1.05x0.95mm_HandSolder" V 7530 2500 50  0001 C CNN
 F 3 "~" H 7600 2500 50  0001 C CNN
 	1    7600 2500
@@
 $EndComp
 $Comp
-L power:GND #PWR?
+L power:GND #PWR0101
 U 1 1 6128E32F
 P 7600 2750
-F 0 "#PWR?" H 7600 2500 50  0001 C CNN
+F 0 "#PWR0101" H 7600 2500 50  0001 C CNN
 F 1 "GND" H 7605 2577 50  0000 C CNN
 F 2 "" H 7600 2750 50  0001 C CNN
@@
 	7450 2300 7600 2300
 Connection ~ 7600 2300
+$Comp
+L Device:LED D19
+U 1 1 60A1DCFB
+P 7550 4200
+F 0 "D19" V 7589 4082 50  0000 R CNN
+F 1 "LED" V 7498 4082 50  0000 R CNN
+F 2 "Robocup_PCB:LED_C210341" H 7550 4200 50  0001 C CNN
+F 3 "~" H 7550 4200 50  0001 C CNN
+	1    7550 4200
+	0    -1   -1   0
+$EndComp
 $EndSCHEMATC

Commit message: update
Parts:
- D1, D10, D11, D12, D13, D14, D15, D16, D17, D18, D19, D2, D20, D21, D22, D23, D24, D3, D4, D5, D6, D7, D8, D9: footprint Robocup_PCB:LED_C210341 -> LED_SMD:LED_0603_1608Metric
- R13, R14, R15, R16, R21, R22, R23, R24, R29, R30, R31, R32, R35, R36, R39, R40, R43, R44, R47, R48, R5, R6, R7, R8: value 62R -> 120R

Commit message: Rounding up main and light board
Parts:
- removed J1: Conn_02x14_Odd_Even, Connector_PinHeader_2.00mm:PinHeader_2x14_P2.00mm_Vertical, symbol Connector_Generic:Conn_02x14_Odd_Even
- removed Q25: 2N7000, Package_TO_SOT_SMD:SOT-223, symbol Transistor_FET:2N7000
- removed R49: 100k, Resistor_SMD:R_0603_1608Metric_Pad1.05x0.95mm_HandSolder, symbol Device:R
- added C?: 0.1u, Capacitor_SMD:C_0603_1608Metric_Pad1.05x0.95mm_HandSolder, symbol Device:C
- added C?: 1u, Capacitor_SMD:C_0603_1608Metric_Pad1.05x0.95mm_HandSolder, symbol Device:C
- added J?: LIGHT_OUT, symbol Connector_Generic:Conn_02x07_Counter_Clockwise
- added Q?: EN, symbol Device:Q_NMOS_GDS
- added R?: 100k, symbol Device:R
- added U1: ADG732, Package_DFN_QFN:QFN-48-1EP_7x7mm_P0.5mm_EP5.15x5.15mm, symbol Main_Board:ADG732
- Q1, Q10, Q11, Q12, Q13, Q14, Q15, Q16, Q17, Q18, Q19, Q2, Q20, Q21, Q22, Q23, Q24, Q3, Q4, Q5, Q6, Q7, Q8, Q9: footprint Robocup_PCB:D_1.70x0.8x0.6mm_handSolder -> Light_Ring:XDCR_ALS-PT19-315C_L177_TR8
- R1, R10, R11, R12, R17, R18, R19, R2, R20, R25, R26, R27, R28, R3, R33, R34, R37, R38, R4, R41, R42, R45, R46, R9: value 22k -> 10k
Connections:
- net +5V: now also C?.1, C?.1, J?.1 (Pin_1), J?.2 (Pin_2), U1.13 (Vdd), U1.14 (Vdd)
- net GND: now also C?.2, C?.2, Q?.3 (S), R?.2, U1.23 (GND), U1.24 (Vss)
- net S1: now also U1.12 (S1)
- net S10: now also U1.3 (S10)
- net S11: now also U1.2 (S11)
- net S12: now also U1.1 (S12)
- net S13: now also U1.48 (S13)
- net S14: now also U1.47 (S14)
- net S15: now also U1.46 (S15)
- net S16: now also U1.45 (S16)
- net S17: now also U1.25 (S17)
- net S18: now also U1.26 (S18)
- net S19: now also U1.27 (S19)
- net S2: now also U1.11 (S2)
- net S20: now also U1.28 (S20)
- net S21: now also U1.29 (S21)
- net S22: now also U1.30 (S22)
- net S23: now also U1.31 (S23)
- net S24: now also U1.32 (S24)
- net S3: now also U1.10 (S3)
- net S4: now also U1.9 (S4)
- net S5: now also U1.8 (S5)
- net S6: now also U1.7 (S6)
- net S7: now also U1.6 (S7)
- net S8: now also U1.5 (S8)
- net S9: now also U1.4 (S9)
- new net: J?.8 (Pin_8), J?.9 (Pin_9), Q?.2 (D)
- new net D: J?.13 (Pin_13), U1.43 (D)
- new net P0: J?.3 (Pin_3), U1.15 (A0)
- new net P1: J?.4 (Pin_4), U1.16 (A1)
- new net P2: J?.5 (Pin_5), U1.17 (A2)
- new net P3: J?.6 (Pin_6), U1.18 (A3)
- new net P4: J?.7 (Pin_7), U1.19 (A4)
- new net PCB_EN: J?.14 (Pin_14), Q?.1 (G), R?.1
- new net ~CS: J?.10 (Pin_10), U1.20 (~CS)
- new net ~EN: J?.12 (Pin_12), U1.22 (~EN)
- new net ~WR: J?.11 (Pin_11), U1.21 (~WR)
- no-connect marks 1 -> 11
Other:
- moved on the sheet: C17, C18, C19, C20, C21, C22, C23, C24, D17, D18, D19, D20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

Commit message: started buck CC driver for LPCB
Parts:
- added U?: LED5000, Package_SO:HSOP-8-1EP_3.9x4.9mm_P1.27mm_EP2.41x3.1mm, symbol Driver_LED:LED5000
Connections:
- new net: U?.6 (GND), U?.9 (GND)
Changed lines of the file:
@@
 Wire Wire Line
 	9350 5650 9350 5900
+$Comp
+L Driver_LED:LED5000 U?
+U 1 1 61F54817
+P 6150 6700
+F 0 "U?" H 6150 7181 50  0000 C CNN
+F 1 "LED5000" H 6150 7090 50  0000 C CNN
+F 2 "Package_SO:HSOP-8-1EP_3.9x4.9mm_P1.27mm_EP2.41x3.1mm" H 6400 6350 50  0001 L CNN
+F 3 "https://www.st.com/resource/en/datasheet/led5000.pdf" H 6050 6350 50  0001 C CNN
+	1    6150 6700
+	1    0    0    -1
+$EndComp
 $EndSCHEMATC

Commit message: Started Light PCB
Parts:
- removed U?: LED5000, Package_SO:HSOP-8-1EP_3.9x4.9mm_P1.27mm_EP2.41x3.1mm, symbol Driver_LED:LED5000
- C1, C10, C11, C12, C13, C14, C15, C16, C17, C18, C19, C2, C20, C21, C22, C23, C24, C3, C4, C5, C6, C7, C8, C9: footprint Capacitor_SMD:C_0603_1608Metric_Pad1.05x0.95mm_HandSolder -> Capacitor_SMD:C_0603_1608Metric_Pad1.08x0.95mm_HandSolder
- C25, C26: renamed from C?; footprint Capacitor_SMD:C_0603_1608Metric_Pad1.05x0.95mm_HandSolder -> Capacitor_SMD:C_0603_1608Metric_Pad1.08x0.95mm_HandSolder
- J1: renamed from J?; footprint (none) -> Connector_JST:JST_PHD_B14B-PHDSS_2x07_P2.00mm_Vertical
- Q25: renamed from Q?; footprint (none) -> Package_TO_SOT_SMD:SOT-23
- R1, R10, R11, R12, R13, R14, R15, R16, R17, R18, R19, R2, R20, R21, R22, R23, R24, R25, R26, R27, R28, R29, R3, R30, R31, R32, R33, R34, R35, R36, R37, R38, R39, R4, R40, R41, R42, R43, R44, R45, R46, R47, R48, R5, R6, R7, R8, R9: footprint Resistor_SMD:R_0603_1608Metric_Pad1.05x0.95mm_HandSolder -> Resistor_SMD:R_0603_1608Metric_Pad0.98x0.95mm_HandSolder
- R49: renamed from R?; footprint (none) -> Resistor_SMD:R_0603_1608Metric_Pad0.98x0.95mm_HandSolder

Commit message: Finished LightPCB
Parts:
- J1: footprint Connector_JST:JST_PHD_B14B-PHDSS_2x07_P2.00mm_Vertical -> Connector_Hirose:Hirose_DF11-14DP-2DSA_2x07_P2.00mm_Vertical
Connections:
- net L16: now reaches U1.29 (S21)
- net L16: now also C16.1, Q16.2 (E), R28.1
- net L12: now reaches U1.33 (S25)
- net L12: now also C12.1, Q12.2 (E), R20.1
- net L11: now reaches U1.34 (S26)
- net L11: now also C11.1, Q11.2 (E), R19.1
- net L10: now reaches U1.35 (S27)
- net L10: now also C10.1, Q10.2 (E), R18.1
- net L9: now reaches U1.36 (S28)
- net L9: now also C9.1, Q9.2 (E), R17.1
- net S1 renamed L1
- net L1: now also U1.8 (S5); no longer U1.12 (S1)
- removed net S10: C10.1, Q10.2 (E), R18.1, U1.3 (S10)
- removed net S11: C11.1, Q11.2 (E), R19.1, U1.2 (S11)
- removed net S12: C12.1, Q12.2 (E), R20.1, U1.1 (S12)
- net S13 renamed L13
- net L13: now also U1.32 (S24); no longer U1.48 (S13)
- net S14 renamed L14
- net L14: now also U1.31 (S23); no longer U1.47 (S14)
- net S15 renamed L15
- net L15: now also U1.30 (S22); no longer U1.46 (S15)
- removed net S16: C16.1, Q16.2 (E), R28.1, U1.45 (S16)
- net S17 renamed L17
- net L17: now also U1.28 (S20); no longer U1.25 (S17)
- net S18 renamed L18
- net L18: now also U1.27 (S19); no longer U1.26 (S18)
- net S19 renamed L19
- net L19: now also U1.26 (S18); no longer U1.27 (S19)
- net S2 renamed L2
- net L2: now also U1.7 (S6); no longer U1.11 (S2)
- net S20 renamed L20
- net L20: now also U1.25 (S17); no longer U1.28 (S20)
- net S21 renamed L21
- net L21: now also U1.12 (S1); no longer U1.29 (S21)
- net S22 renamed L22
- net L22: now also U1.11 (S2); no longer U1.30 (S22)
- net S23 renamed L23
- net L23: now also U1.10 (S3); no longer U1.31 (S23)
- net S24 renamed L24
- net L24: now also U1.9 (S4); no longer U1.32 (S24)
- net S3 renamed L3
- net L3: now also U1.6 (S7); no longer U1.10 (S3)
- net S4 renamed L4
- net L4: now also U1.5 (S8); no longer U1.9 (S4)
- net S5 renamed L5
- net L5: now also U1.4 (S9); no longer U1.8 (S5)
- net S6 renamed L6
- net L6: now also U1.3 (S10); no longer U1.7 (S6)
- net S7 renamed L7
- net L7: now also U1.2 (S11); no longer U1.6 (S7)
- net S8 renamed L8
- net L8: now also U1.1 (S12); no longer U1.5 (S8)
- removed net S9: C9.1, Q9.2 (E), R17.1, U1.4 (S9)
- net ~CS renamed ~CL
Changed lines of the file:
@@
 	9950 2800 9950 3050
 Text GLabel 1350 1350 2    50   Output ~ 0
-S1
+L1
 Text GLabel 1350 3000 2    50   Output ~ 0
-S2
+L2
 Text GLabel 1350 4650 2    50   Output ~ 0
-S3
+L3
 Text GLabel 1350 6300 2    50   Output ~ 0
-S4
+L4
 Text GLabel 2550 1350 2    50   Output ~ 0
-S5
+L5
 Text GLabel 2550 3000 2    50   Output ~ 0
-S6
+L6
 Text GLabel 2550 4650 2    50   Output ~ 0
-S7
+L7
 Text GLabel 2550 6300 2    50   Output ~ 0
-S8
+L8
 Text GLabel 3700 1300 2    50   Output ~ 0
-S9
+L9
 Text GLabel 3700 2950 2    50   Output ~ 0
-S10
+L10
 Text GLabel 3700 4600 2    50   Output ~ 0
-S11
+L11
 Text GLabel 3700 6250 2    50   Output ~ 0
-S12
+L12
 Text GLabel 4900 1300 2    50   Output ~ 0
-S13
+L13
 Text GLabel 4900 2950 2    50   Output ~ 0
-S14
+L14
 Text GLabel 4900 4600 2    50   Output ~ 0
-S15
+L15
 Text GLabel 4900 6250 2    50   Output ~ 0
-S16
+L16
 Text GLabel 6100 1300 2    50   Output ~ 0
-S17
+L17
 Text GLabel 6100 2950 2    50   Output ~ 0
-S18
+L18
 Text GLabel 7300 1300 2    50   Output ~ 0
-S19
+L19
 Text GLabel 7300 2950 2    50   Output ~ 0
-S20
+L20
 Text GLabel 8500 1300 2    50   Output ~ 0
-S21
+L21
 Text GLabel 8500 2950 2    50   Output ~ 0
-S22
+L22
 Text GLabel 9700 1300 2    50   Output ~ 0
-S23
+L23
 Text GLabel 9700 2950 2    50   Output ~ 0
-S24
+L24
+Text GLabel 8200 5000 0    50   Input ~ 0
+L1
+Text GLabel 8200 4300 0    50   Input ~ 0
+L8
+Text GLabel 10200 4600 2    50   Input ~ 0
+L12
+Text GLabel 10200 4500 2    50   Input ~ 0
+L11
+Text GLabel 10200 4400 2    50   Input ~ 0
+L10
+Text GLabel 10200 4300 2    50   Input ~ 0
+L9
+Text GLabel 8200 4400 0    50   Input ~ 0
+L7
+Text GLabel 8200 4500 0    50   Input ~ 0
+L6
+Text GLabel 8200 4600 0    50   Input ~ 0
+L5
+Text GLabel 8200 4700 0    50   Input ~ 0
+L4
+Text GLabel 8200 4900 0    50   Input ~ 0
+L2
+Text GLabel 10200 4700 2    50   Input ~ 0
+L13
+Text GLabel 10200 4800 2    50   Input ~ 0
+L14
+Text GLabel 10200 4900 2    50   Input ~ 0
+L15
+Text GLabel 10200 5000 2    50   Input ~ 0
+L16
+Text GLabel 10200 5100 2    50   Input ~ 0
+L17
+Text GLabel 10200 5200 2    50   Input ~ 0
+L18
+Text GLabel 10200 5400 2    50   Input ~ 0
+L20
+Text GLabel 8200 5300 0    50   Input ~ 0
+L22
+Text GLabel 8200 5200 0    50   Input ~ 0
+L23
 Text GLabel 8200 5400 0    50   Input ~ 0
-S1
-Text GLabel 8200 4700 0    50   Input ~ 0
-S8
-Text GLabel 8200 4300 0    50   Input ~ 0
-S12
-Text GLabel 8200 4400 0    50   Input ~ 0
-S11
-Text GLabel 8200 4500 0    50   Input ~ 0
-S10
-Text GLabel 8200 4600 0    50   Input ~ 0
-S9
-Text GLabel 8200 4800 0    50   Input ~ 0
-S7
-Text GLabel 8200 4900 0    50   Input ~ 0
-S6
-Text GLabel 8200 5000 0    50   Input ~ 0
-S5
-Text GLabel 8200 5100 0    50   Input ~ 0
-S4
-Text GLabel 8200 5200 0    50   Input ~ 0
-S3
-Text GLabel 8200 5300 0    50   Input ~ 0
-S2
-Text GLabel 8650 3950 1    50   Input ~ 0
-S13
-Text GLabel 8750 3950 1    50   Input ~ 0
-S14
-Text GLabel 8850 3950 1    50   Input ~ 0
-S15
-Text GLabel 8950 3950 1    50   Input ~ 0
-S16
-Text GLabel 10200 5400 2    50   Input ~ 0
-S17
+L21
 Text GLabel 10200 5300 2    50   Input ~ 0
-S18
-Text GLabel 10200 5100 2    50   Input ~ 0
-S20
-Text GLabel 10200 4900 2    50   Input ~ 0
-S22
-Text GLabel 10200 4700 2    50   Input ~ 0
-S24
-Text GLabel 10200 4800 2    50   Input ~ 0
-S23
-Text GLabel 10200 5000 2    50   Input ~ 0
-S21
-Text GLabel 10200 5200 2    50   Input ~ 0
-S19
+L19
 $Comp
 L Device:LED D19
@@
 	0    -1   -1   0
 $EndComp
-$Comp
-L Main_Board:ADG732 U1
-U 1 1 61F76C65
-P 9200 4850
-F 0 "U1" H 8400 5600 50  0000 L CNN
-F 1 "ADG732" H 9050 4850 50  0000 L CNN
-F 2 "Package_DFN_QFN:QFN-48-1EP_7x7mm_P0.5mm_EP5.15x5.15mm" H 9700 3850 50  0001 C CNN
-F 3 "https://www.analog.com/media/en/technical-documentation/data-sheets/adg726_732.pdf" H 8700 5250 50  0001 C CNN
-	1    9200 4850
-	1    0    0    -1
-$EndComp
-Wire Wire Line
-	8200 5400 8300 5400
-Wire Wire Line
-	8200 5300 8300 5300
-Wire Wire Line
-	8200 5200 8300 5200
-Wire Wire Line
-	8200 5100 8300 5100
-Wire Wire Line
-	8200 5000 8300 5000
-Wire Wire Line
-	8200 4900 8300 4900
-Wire Wire Line
-	8200 4800 8300 4800
-Wire Wire Line
-	8200 4700 8300 4700
-Wire Wire Line
-	8200 4600 8300 4600
-Wire Wire Line
-	8200 4500 8300 4500
-Wire Wire Line
-	8200 4400 8300 4400
-Wire Wire Line
-	8200 4300 8300 4300
-Wire Wire Line
-	8650 3950 8650 4050
-Wire Wire Line
-	8750 3950 8750 4050
-Wire Wire Line
-	8850 3950 8850 4050
-Wire Wire Line
-	8950 3950 8950 4050
-Wire Wire Line
-	10200 4700 10100 4700
-Wire Wire Line
-	10200 4800 10100 4800
-Wire Wire Line
-	10200 4900 10100 4900
-Wire Wire Line
-	10200 5000 10100 5000
-Wire Wire Line
-	10200 5100 10100 5100
-Wire Wire Line
-	10200 5200 10100 5200
-Wire Wire Line
-	10200 5300 10100 5300
-Wire Wire Line
-	10200 5400 10100 5400
 NoConn ~ 9050 4050
 NoConn ~ 9250 4050
 NoConn ~ 9350 4050
-NoConn ~ 9450 4050
-NoConn ~ 9550 4050
-NoConn ~ 9650 4050
-NoConn ~ 9750 4050
-NoConn ~ 10100 4600
-NoConn ~ 10100 4500
-NoConn ~ 10100 4400
-NoConn ~ 10100 4300
 $Comp
 L Device:C C26
@@
 F 0 "J1" V 7100 4700 50  0000 R CNN
 F 1 "LIGHT_OUT" V 7100 5250 50  0000 R CNN
-F 2 "Connector_JST:JST_PHD_B14B-PHDSS_2x07_P2.00mm_Vertical" H 7050 4950 50  0001 C CNN
+F 2 "Connector_Hirose:Hirose_DF11-14DP-2DSA_2x07_P2.00mm_Vertical" H 7050 4950 50  0001 C CNN
 F 3 "~" H 7050 4950 50  0001 C CNN
 	1    7050 4950
@@
 ~WR
 Text GLabel 7600 5050 2    50   Output ~ 0
-~CS
+~CL
 Wire Wire Line
 	7450 4950 7350 4950
@@
 ~WR
 Text GLabel 9350 5900 3    50   Input ~ 0
-~CS
+~CL
 Wire Wire Line
 	9750 5850 9750 5750
@@
 Wire Wire Line
 	9350 5650 9350 5900
+Text GLabel 8200 5100 0    50   Input ~ 0
+L24
+$Comp
+L Main_Board:ADG732 U1
+U 1 1 61F76C65
+P 9200 4850
+F 0 "U1" H 8400 5600 50  0000 L CNN
+F 1 "ADG732" H 9050 4850 50  0000 L CNN
+F 2 "Package_DFN_QFN:QFN-48-1EP_7x7mm_P0.5mm_EP5.15x5.15mm" H 9700 3850 50  0001 C CNN
+F 3 "https://www.analog.com/media/en/technical-documentation/data-sheets/adg726_732.pdf" H 8700 5250 50  0001 C CNN
+	1    9200 4850
+	1    0    0    -1
+$EndComp
+Text GLabel 8200 4800 0    50   Input ~ 0
+L3
+Wire Wire Line
+	8200 5400 8300 5400
+Wire Wire Line
+	8200 5300 8300 5300
+Wire Wire Line
+	8200 5200 8300 5200
+Wire Wire Line
+	8200 5100 8300 5100
+Wire Wire Line
+	8200 5000 8300 5000
+Wire Wire Line
+	8200 4900 8300 4900
+Wire Wire Line
+	8200 4800 8300 4800
+Wire Wire Line
+	8200 4700 8300 4700
+Wire Wire Line
+	8200 4600 8300 4600
+Wire Wire Line
+	8200 4500 8300 4500
+Wire Wire Line
+	8200 4400 8300 4400
+Wire Wire Line
+	8200 4300 8300 4300
+NoConn ~ 8650 4050
+NoConn ~ 8750 4050
+NoConn ~ 8850 4050
+NoConn ~ 8950 4050
+NoConn ~ 9450 4050
+NoConn ~ 9550 4050
+NoConn ~ 9650 4050
+NoConn ~ 9750 4050
+Wire Wire Line
+	10100 4300 10200 4300
+Wire Wire Line
+	10200 4400 10100 4400
+Wire Wire Line
+	10100 4500 10200 4500
+Wire Wire Line
+	10200 4600 10100 4600
+Wire Wire Line
+	10100 4700 10200 4700
+Wire Wire Line
+	10200 4800 10100 4800
+Wire Wire Line
+	10100 4900 10200 4900
+Wire Wire Line
+	10200 5000 10100 5000
+Wire Wire Line
+	10100 5100 10200 5100
+Wire Wire Line
+	10200 5200 10100 5200
+Wire Wire Line
+	10100 5300 10200 5300
+Wire Wire Line
+	10200 5400 10100 5400
 $EndSCHEMATC
