File: Light_Ring_PCB/Light_Ring_PCB.sch (KiCad schematic (older format))
At the start: 126 parts, among them J1 LIGHT_OUT, Q1 Q_Photo_NPN, Q10 Q_Photo_NPN, Q11 Q_Photo_NPN, Q12 Q_Photo_NPN, Q13 Q_Photo_NPN, Q14 Q_Photo_NPN, Q15 Q_Photo_NPN, Q16 Q_Photo_NPN, Q17 Q_Photo_NPN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

Commit message: Finished Main PCB schematic
Parts:
- R1, R10, R11, R12, R17, R18, R19, R2, R20, R25, R26, R27, R28, R3, R33, R34, R37, R38, R4, R41, R42, R45, R46, R9: value 10k -> 6k2
- R13, R14, R15, R16, R21, R22, R23, R24, R29, R30, R31, R32, R35, R36, R39, R40, R43, R44, R47, R48, R5, R6, R7, R8: value 120R -> 12R
Connections:
- net +5V renamed +3V3
Other:
- note added: "IF Vf = 3.1V, then Rled = 12R\nIF Vf = 2.9V, then Rled = 25R"

Commit message: Finished Power Planes and layout, started drawing traces [MAIN BOARD]
Parts:
- U1: footprint Package_DFN_QFN:QFN-48-1EP_7x7mm_P0.5mm_EP5.15x5.15mm -> Package_CSP:LFCSP-48-1EP_7x7mm_P0.5mm_EP4.1x4.1mm
Changed lines of the file:
@@
 F 0 "U1" H 8400 5600 50  0000 L CNN
 F 1 "ADG732" H 9050 4850 50  0000 L CNN
-F 2 "Package_DFN_QFN:QFN-48-1EP_7x7mm_P0.5mm_EP5.15x5.15mm" H 9700 3850 50  0001 C CNN
+F 2 "Package_CSP:LFCSP-48-1EP_7x7mm_P0.5mm_EP4.1x4.1mm" H 9700 3850 50  0001 C CNN
 F 3 "https://www.analog.com/media/en/technical-documentation/data-sheets/adg726_732.pdf" H 8700 5250 50  0001 C CNN
 	1    9200 4850
