File: Light_Ring_PCB/Light_Ring_PCB.kicad_pcb (KiCad board)
At the start: 2 copper layers, 123 parts, among them J1 Conn_02x14_Odd_Even, Q1 Q_Photo_NPN, Q10 Q_Photo_NPN, Q11 Q_Photo_NPN, Q12 Q_Photo_NPN, Q13 Q_Photo_NPN, Q14 Q_Photo_NPN, Q15 Q_Photo_NPN, Q16 Q_Photo_NPN, Q17 Q_Photo_NPN, Q18 Q_Photo_NPN, Q19 Q_Photo_NPN, Q2 Q_Photo_NPN, Q20 Q_Photo_NPN, Q21 Q_Photo_NPN, Q22 Q_Photo_NPN, Q23 Q_Photo_NPN, Q24 Q_Photo_NPN, Q25 2N7000, Q3 Q_Photo_NPN, Q4 Q_Photo_NPN, Q5 Q_Photo_NPN, Q6 Q_Photo_NPN, Q7 Q_Photo_NPN, Q8 Q_Photo_NPN, Q9 Q_Photo_NPN

Commit message: Started PCB
Parts:
- moved Q25 131.6 mm to (136.6, 156.4), turned to 270 degrees
- moved J1 112.6 mm to (134.9, 124.0)
- moved Q1 98.3 mm to (49.8, 143.6)
- moved Q10 98.3 mm to (57.7, 141.1)
- moved Q11 98.3 mm to (55.8, 136.1)
- moved Q12 98.3 mm to (54.2, 138.7)
- moved Q16 98.3 mm to (50.3, 138.7)
- moved Q17 98.3 mm to (45.9, 143.6)
- moved Q2 98.3 mm to (53.7, 141.1)
- moved Q23 98.3 mm to (41.5, 146.2)
- moved Q8 98.3 mm to (53.7, 143.5)
- moved Q13 98.3 mm to (49.8, 141.2)
- moved Q15 98.3 mm to (45.9, 141.2)
- moved Q18 98.3 mm to (55.8, 133.7)
- moved Q24 98.3 mm to (45.9, 146.0)
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Other:
- board outline added: 209.7 x 196.1 mm

Commit message: update
Parts:
- D1, D10, D11, D12, D13, D14, D15, D16, D17, D18, D19, D2, D20, D21, D22, D23, D24, D3, D4, D5, D6, D7, D8, D9: footprint Robocup_PCB:LED_C210341 -> LED_SMD:LED_0603_1608Metric
- R13, R14, R15, R16, R21, R22, R23, R24, R29, R30, R31, R32, R35, R36, R39, R40, R43, R44, R47, R48, R5, R6, R7, R8: value 62R -> 120R
- moved D13 229.4 mm to (229.1, 231.6), turned to 90 degrees
- moved D20 219.1 mm to (247.0, 136.5)
- moved D11 218.9 mm to (246.7, 139.1)
- moved C14 212.9 mm to (211.4, 231.6), turned to 90 degrees
- moved D14 212.8 mm to (205.0, 231.6), turned to 90 degrees
- moved D24 206.1 mm to (228.4, 151.5)
- moved D17 205.9 mm to (236.8, 146.5)
- moved Q5 205.9 mm to (248.7, 146.5)
- moved D22 204.8 mm to (232.8, 146.5)
- moved D18 204.0 mm to (228.4, 154.1)
- moved D16 203.3 mm to (232.8, 149.1)
- moved Q13 203.3 mm to (231.9, 231.6), turned to 90 degrees
- moved Q21 201.9 mm to (244.8, 144.2)
- moved D23 201.2 mm to (224.1, 156.6)
- moved D19 200.4 mm to (224.1, 159.2)
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Routing:
- net S14: track 0.00 -> 3.61 mm
- net +5V: track 0.00 -> 2.16 mm
- net Net-(D14-Pad2): track 0.00 -> 1.81 mm
Other:
- rule trace_min: 0.2 -> 0.127
- rule via_min_size: 0.4 -> 0.6

Commit message: Yes
Other:
- board outline removed

Commit message: Rounding up main and light board
Parts:
- Q1, Q10, Q11, Q12, Q13, Q14, Q15, Q16, Q17, Q18, Q19, Q2, Q20, Q21, Q22, Q23, Q24, Q3, Q4, Q5, Q6, Q7, Q8, Q9: footprint Robocup_PCB:D_1.70x0.8x0.6mm_handSolder -> Light_Ring:XDCR_ALS-PT19-315C_L177_TR8
- R1, R10, R11, R12, R17, R18, R19, R2, R20, R25, R26, R27, R28, R3, R33, R34, R37, R38, R4, R41, R42, R45, R46, R9: value 22k -> 10k
- moved Q14 108.7 mm to (209.4, 122.9), turned to 0 degrees
- moved R14 107.3 mm to (242.9, 118.3)
- moved Q13 103.3 mm to (199.6, 133.5), turned to 0 degrees
- moved R26 102.0 mm to (225.5, 130.8), turned to 0 degrees
- moved C14 101.5 mm to (216.8, 130.2), turned to 0 degrees
- moved D14 99.9 mm to (234.0, 136.0), turned to 0 degrees
- moved D13 85.7 mm to (223.6, 146.0), turned to 0 degrees
- moved R30 81.8 mm to (215.0, 147.8), turned to 0 degrees
- moved R13 79.0 mm to (221.0, 138.0)
- moved Q12 55.2 mm to (193.5, 148.3)
- moved R19 54.3 mm to (238.6, 118.3)
- moved R8 52.4 mm to (235.3, 120.8)
- moved C3 52.2 mm to (234.2, 118.3)
- moved R3 51.8 mm to (239.6, 120.8)
- moved R37 48.7 mm to (244.0, 120.8)
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Connections:
- J1 pad 26: Net-(J1-Pad26) -> +5V
Routing:
- net S14: track 3.61 -> 0.00 mm
- net +5V: track 2.16 -> 0.00 mm
- net Net-(D14-Pad2): track 1.81 -> 0.00 mm

Commit message: Started Light PCB
Parts:
- added C25: 1u, Capacitor_SMD:C_0603_1608Metric_Pad1.08x0.95mm_HandSolder, F.Cu at (118.4, 129.5)
- added C26: 0.1u, Capacitor_SMD:C_0603_1608Metric_Pad1.08x0.95mm_HandSolder, F.Cu at (122.0, 139.5)
- added U1: ADG732, Package_DFN_QFN:QFN-48-1EP_7x7mm_P0.5mm_EP5.15x5.15mm, F.Cu at (207.3, 123.4)
- C1, C10, C11, C12, C13, C14, C15, C16, C17, C18, C19, C2, C20, C21, C22, C23, C24, C3, C4, C5, C6, C7, C8, C9: footprint Capacitor_SMD:C_0603_1608Metric_Pad1.05x0.95mm_HandSolder -> Capacitor_SMD:C_0603_1608Metric_Pad1.08x0.95mm_HandSolder
- J1: value Conn_02x14_Odd_Even -> LIGHT_OUT; footprint Connector_PinHeader_2.00mm:PinHeader_2x14_P2.00mm_Vertical -> Connector_JST:JST_PHD_B14B-PHDSS_2x07_P2.00mm_Vertical
- Q25: value 2N7000 -> EN; footprint Package_TO_SOT_SMD:SOT-223 -> Package_TO_SOT_SMD:SOT-23
- R1, R10, R11, R12, R13, R14, R15, R16, R17, R18, R19, R2, R20, R21, R22, R23, R24, R25, R26, R27, R28, R29, R3, R30, R31, R32, R33, R34, R35, R36, R37, R38, R39, R4, R40, R41, R42, R43, R44, R45, R46, R47, R48, R49, R5, R6, R7, R8, R9: footprint Resistor_SMD:R_0603_1608Metric_Pad1.05x0.95mm_HandSolder -> Resistor_SMD:R_0603_1608Metric_Pad0.98x0.95mm_HandSolder
- moved R49 110.0 mm to (121.5, 133.5)
- moved D19 91.3 mm to (151.5, 127.5), turned to 359 degrees
- moved R37 89.4 mm to (155.0, 129.4), turned to 1 degrees
- moved R39 89.1 mm to (155.0, 127.6), turned to 179 degrees
- moved D21 85.5 mm to (159.3, 100.2), turned to 329 degrees
- moved D23 84.0 mm to (179.8, 80.4), turned to 299 degrees
- moved D17 83.6 mm to (158.4, 155.1), turned to 29 degrees
- moved D20 82.9 mm to (153.6, 113.3), turned to 344 degrees
- moved D22 81.9 mm to (168.2, 89.0), turned to 314 degrees
- moved R43 80.6 mm to (162.3, 102.0), turned to 149 degrees
- moved R32 79.1 mm to (169.4, 164.2), turned to 224 degrees
- moved D18 76.6 mm to (153.1, 141.8), turned to 14 degrees
- moved R35 76.2 mm to (161.4, 153.4), turned to 209 degrees
- moved R38 75.9 mm to (156.5, 116.0), turned to 346 degrees
- moved D24 75.6 mm to (193.1, 75.2), turned to 284 degrees
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Connections:
- J1 pad 1: S1 -> +5V
- J1 pad 10: S10 -> ~CS
- J1 pad 11: S11 -> ~WR
- J1 pad 12: S12 -> ~EN
- J1 pad 13: S13 -> D
- J1 pad 14: S14 -> PCB_EN
- J1 pad 2: S2 -> +5V
- J1 pad 3: S3 -> P0
- J1 pad 4: S4 -> P1
- J1 pad 5: S5 -> P2
- J1 pad 6: S6 -> P3
- J1 pad 7: S7 -> P4
- J1 pad 8: S8 -> Net-(J1-Pad8)
- J1 pad 9: S9 -> Net-(J1-Pad8)
- Q25 pad 1: GND -> PCB_EN
- Q25 pad 2: EN -> Net-(J1-Pad8)
- Q25 pad 3: Net-(J1-Pad27) -> GND
- R49 pad 1: EN -> PCB_EN
Routing:
- net S8: track 0.00 -> 70.8 mm
- net S7: track 0.00 -> 66.6 mm
- net S5: track 0.00 -> 62.0 mm
- net S6: track 0.00 -> 59.7 mm
- net S4: track 0.00 -> 58.1 mm
- net S3: track 0.00 -> 52.7 mm
- net S2: track 0.00 -> 52.3 mm
- net S1: track 0.00 -> 47.9 mm
- net S9: track 0.00 -> 3.93 mm
- net S12: track 0.00 -> 3.93 mm
- net S18: track 0.00 -> 3.93 mm
- net S23: track 0.00 -> 3.89 mm
- net S17: track 0.00 -> 3.89 mm
- net S11: track 0.00 -> 3.89 mm
- net S20: track 0.00 -> 3.89 mm
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Other:
- board outline added: 120 x 120 mm

Commit message: Finished LightPCB
Parts:
- J1: footprint Connector_JST:JST_PHD_B14B-PHDSS_2x07_P2.00mm_Vertical -> Connector_Hirose:Hirose_DF11-14DP-2DSA_2x07_P2.00mm_Vertical; moved to B.Cu
- Q25, R49: moved to B.Cu
- moved C25 90.6 mm to (208.7, 121.6), turned to 90 degrees
- moved C26 86.9 mm to (207.0, 121.6), turned to 90 degrees
- moved R49 86.2 mm to (207.6, 130.5)
- moved Q25 79.8 mm to (207.6, 133.5)
- moved J1 21.7 mm to (201.7, 122.4), turned to 270 degrees
- moved U1 8.45 mm to (214.4, 127.9)
Connections:
- net ~CS renamed ~CL
- C1 pad 1: S1 -> L1
- C10 pad 1: S10 -> L10
- C11 pad 1: S11 -> L11
- C12 pad 1: S12 -> L12
- C13 pad 1: S13 -> L13
- C14 pad 1: S14 -> L14
- C15 pad 1: S15 -> L15
- C16 pad 1: S16 -> L16
- C17 pad 1: S17 -> L17
- C18 pad 1: S18 -> L18
- C19 pad 1: S19 -> L19
- C2 pad 1: S2 -> L2
- C20 pad 1: S20 -> L20
- C21 pad 1: S21 -> L21
- C22 pad 1: S22 -> L22
- C23 pad 1: S23 -> L23
- C24 pad 1: S24 -> L24
- C3 pad 1: S3 -> L3
- C4 pad 1: S4 -> L4
- C5 pad 1: S5 -> L5
- C6 pad 1: S6 -> L6
- C7 pad 1: S7 -> L7
- C8 pad 1: S8 -> L8
- C9 pad 1: S9 -> L9
- Q1 pad 2: S1 -> L1
- Q10 pad 2: S10 -> L10
- Q11 pad 2: S11 -> L11
- Q12 pad 2: S12 -> L12
- Q13 pad 2: S13 -> L13
- Q14 pad 2: S14 -> L14
- Q15 pad 2: S15 -> L15
- Q16 pad 2: S16 -> L16
- Q17 pad 2: S17 -> L17
- Q18 pad 2: S18 -> L18
- Q19 pad 2: S19 -> L19
- Q2 pad 2: S2 -> L2
- Q20 pad 2: S20 -> L20
- Q21 pad 2: S21 -> L21
- Q22 pad 2: S22 -> L22
- Q23 pad 2: S23 -> L23
- Q24 pad 2: S24 -> L24
- Q3 pad 2: S3 -> L3
- Q4 pad 2: S4 -> L4
- Q5 pad 2: S5 -> L5
- Q6 pad 2: S6 -> L6
- Q7 pad 2: S7 -> L7
- Q8 pad 2: S8 -> L8
- Q9 pad 2: S9 -> L9
- R1 pad 1: S1 -> L1
- R10 pad 1: S6 -> L6
- R11 pad 1: S7 -> L7
- R12 pad 1: S8 -> L8
- R17 pad 1: S9 -> L9
- R18 pad 1: S10 -> L10
- R19 pad 1: S11 -> L11
- R2 pad 1: S2 -> L2
- R20 pad 1: S12 -> L12
- R25 pad 1: S13 -> L13
- R26 pad 1: S14 -> L14
- R27 pad 1: S15 -> L15
- R28 pad 1: S16 -> L16
- R3 pad 1: S3 -> L3
- R33 pad 1: S17 -> L17
- R34 pad 1: S18 -> L18
- R37 pad 1: S19 -> L19
- R38 pad 1: S20 -> L20
- R4 pad 1: S4 -> L4
- R41 pad 1: S21 -> L21
- R42 pad 1: S22 -> L22
- R45 pad 1: S23 -> L23
- R46 pad 1: S24 -> L24
- R9 pad 1: S5 -> L5
- U1 pad 1: S12 -> L8
- U1 pad 10: S3 -> L23
- U1 pad 11: S2 -> L22
- U1 pad 12: S1 -> L21
- U1 pad 2: S11 -> L7
- U1 pad 25: S17 -> L20
- U1 pad 26: S18 -> L19
- U1 pad 27: S19 -> L18
- U1 pad 28: S20 -> L17
- U1 pad 29: S21 -> L16
- U1 pad 3: S10 -> L6
- U1 pad 30: S22 -> L15
- U1 pad 31: S23 -> L14
- U1 pad 32: S24 -> L13
- U1 pad 33: Net-(U1-Pad33) -> L12
- U1 pad 34: Net-(U1-Pad34) -> L11
- U1 pad 35: Net-(U1-Pad35) -> L10
- U1 pad 36: Net-(U1-Pad36) -> L9
- U1 pad 4: S9 -> L5
- U1 pad 45: S16 -> Net-(U1-Pad45)
- U1 pad 46: S15 -> Net-(U1-Pad46)
- U1 pad 47: S14 -> Net-(U1-Pad47)
- U1 pad 48: S13 -> Net-(U1-Pad48)
- U1 pad 49: (no net) -> GND
- U1 pad 5: S8 -> L4
- U1 pad 6: S7 -> L3
- U1 pad 7: S6 -> L2
- U1 pad 8: S5 -> L1
- U1 pad 9: S4 -> L24
Routing:
- net GND: track 0.00 -> 183.8 mm, vias 0 -> 73
- net L20: track 0.00 -> 87.6 mm
- net L19: track 0.00 -> 81.6 mm
- net L16: track 0.00 -> 77.6 mm
- net L18: track 0.00 -> 74.7 mm
- net L15: track 0.00 -> 73.6 mm
- net L17: track 0.00 -> 73.1 mm
- net S8: track 70.8 -> 0.00 mm
- net S7: track 66.6 -> 0.00 mm
- net L21: track 0.00 -> 65.2 mm
- net L14: track 0.00 -> 62.7 mm
- net S5: track 62.0 -> 0.00 mm
- net L11: track 0.00 -> 61.1 mm
- net L22: track 0.00 -> 61.0 mm
- net S6: track 59.7 -> 0.00 mm
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- added copper zone on F.Cu, net +5V
- added copper zone on B.Cu, net GND
Other:
- rule via_min_drill: 0.3 -> 0.2
- rule via_min_size: 0.6 -> 0.4

Commit message: Finished Light PCB
Parts:
- C25, C26: moved to B.Cu
- moved R49 12.5 mm to (210.1, 142.7)
- moved C26 9.93 mm to (211.3, 130.5)
- moved C25 9.01 mm to (209.7, 130.5)
- moved J1 7.50 mm to (204.1, 129.5)
- moved Q25 7.11 mm to (210.1, 140.2)
- moved C10 6.48 mm to (243.4, 169.2)
- moved C13 6.48 mm to (207.8, 186.2)
- moved C9 6.48 mm to (251.0, 158.2)
- moved D12 6.48 mm to (218.4, 188.1)
- moved Q11 6.48 mm to (233.4, 181.9)
- moved Q14 6.48 mm to (191.8, 188.1)
- moved Q18 6.48 mm to (152.3, 150.0)
- moved Q19 6.48 mm to (150.2, 135.8)
- moved R21 6.48 mm to (249.2, 161.3)
- moved R25 6.48 mm to (206.0, 186.3)
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Connections:
- J1 pad 3: P0 -> P1
- J1 pad 4: P1 -> P0
- J1 pad 5: P2 -> P3
- J1 pad 6: P3 -> P2
Routing:
- net +5V: track 42.2 -> 29.2 mm, vias 16 -> 10
- net GND: track 183.8 -> 177.0 mm, vias 73 -> 72
- net P2: track 10.1 -> 3.61 mm, vias 1 -> 0
- net L2: track 58.8 -> 52.6 mm
- net P0: track 10.1 -> 4.03 mm, vias 1 -> 0
- net PCB_EN: track 9.77 -> 4.76 mm
- net D: track 24.5 -> 21.3 mm
- net P4: track 10.3 -> 7.26 mm, vias 1 -> 0
- net ~CL: track 7.95 -> 5.08 mm
- net L1: track 55.5 -> 58.1 mm
- net ~WR: track 10.6 -> 8.37 mm
- net ~EN: track 8.37 -> 6.27 mm
- net P1: track 8.23 -> 6.73 mm, vias 1 -> 0
- net P3: track 7.82 -> 6.63 mm
- net L23: track 58.9 -> 58.2 mm, vias 2 -> 0
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Other:
- outline, holes or cut-outs redrawn
- board text added: "Goaly Light Ring Module v1.2 Designed by Pixeljoch, January 2022 Funded by Leaphy"
- board text added: "niet aan likken a.u.b."
