File: Main_Board/Main_Board.kicad_pcb (KiCad board)
At the start: 4 copper layers, 120 x 140 mm, 67 parts, among them J1 Conn_01x06, J10 HR-SR04_L_CONN, J11 12V_OUT, J12 BATT_REG_IN, J13 LED_CONN, J14 PD_CONN, J2 Conn_01x06, J3 Conn_01x06, J4 BATT_IN, J5 Conn_02x08_Top_Bottom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

Commit message: Finished board [MAIN BOARD]
Parts:
- added 12V: TestPoint_Pad_D1.0mm, TestPoint:TestPoint_Pad_D1.0mm, F.Cu at (177.3, 73.2)
- added 3.3V: TestPoint_Pad_D1.0mm, TestPoint:TestPoint_Pad_D1.0mm, F.Cu at (144.0, 83.8)
- added ECHO_L: TestPoint_Pad_D1.0mm, TestPoint:TestPoint_Pad_D1.0mm, F.Cu at (203.5, 96.8)
- added ECHO_R: TestPoint_Pad_D1.0mm, TestPoint:TestPoint_Pad_D1.0mm, F.Cu at (99.6, 100.8)
- added M1_PWM: TestPoint_Pad_D1.0mm, TestPoint:TestPoint_Pad_D1.0mm, F.Cu at (184.2, 154.1)
- added M2_PWM: TestPoint_Pad_D1.0mm, TestPoint:TestPoint_Pad_D1.0mm, F.Cu at (106.7, 153.9)
- added M3_PWM: TestPoint_Pad_D1.0mm, TestPoint:TestPoint_Pad_D1.0mm, F.Cu at (201.9, 116.8)
- added M4: MountingHole_4.3mm_M4, MountingHole:MountingHole_4.3mm_M4, F.Cu at (204.2, 154.7)
- added M4: MountingHole_4.3mm_M4, MountingHole:MountingHole_4.3mm_M4, F.Cu at (94.3, 154.7)
- added REF**: OSHW-Symbol_6.7x6mm_SilkScreen, Symbol:OSHW-Symbol_6.7x6mm_SilkScreen, B.Cu at (142.0, 155.2)
- added REF**: MountingHole_4.3mm_M4, MountingHole:MountingHole_4.3mm_M4, F.Cu at (149.3, 124.9)
- added REF**: MountingHole_4.3mm_M4, MountingHole:MountingHole_4.3mm_M4, F.Cu at (129.3, 24.9)
- added REF**: MountingHole_4.3mm_M4, MountingHole:MountingHole_4.3mm_M4, F.Cu at (169.3, 24.9)
- added TRIG_L: TestPoint_Pad_D1.0mm, TestPoint:TestPoint_Pad_D1.0mm, F.Cu at (205.7, 96.8)
- added TRIG_R: TestPoint_Pad_D1.0mm, TestPoint:TestPoint_Pad_D1.0mm, F.Cu at (99.6, 104.6)
- added VBAT: TestPoint_Pad_D1.0mm, TestPoint:TestPoint_Pad_D1.0mm, F.Cu at (138.2, 57.9)
- moved R2 3.85 mm to (156.2, 58.8)
Connections:
- J4 pad 1: GND -> Net-(J4-Pad2)
- J4 pad 2: Net-(J4-Pad2) -> GND
- U1 pad 3.3V_1: Net-(U1-Pad3.3V_1) -> (no net)
- U2 pad 3.3V_1: Net-(U2-Pad3.3V_1) -> (no net)
Routing:
- net M3_PWM: track 46.6 -> 65.4 mm, vias 0 -> 1
- net TRIG_L: track 88.4 -> 97.4 mm
- net GND: track 85.9 -> 94.3 mm, vias 20 -> 26
- net ECHO_R: track 33.0 -> 39.5 mm
- net ECHO_L: track 91.2 -> 97.3 mm
- net TRIG_R: track 34.8 -> 40.7 mm
- net M1_PWM: track 48.4 -> 53.6 mm
- net M2_PWM: track 23.5 -> 28.6 mm
- net ~EN: track 6.84 -> 11.2 mm
- net +3V3: track 61.5 -> 65.0 mm
- net ~WR: track 10.7 -> 13.3 mm
- net P0: track 7.24 -> 9.91 mm
- net P4: track 16.7 -> 18.8 mm
- net +VDC: track 16.1 -> 14.2 mm, vias 43 -> 40
- net ~CS: track 11.3 -> 12.8 mm
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Other:
- outline, holes or cut-outs redrawn
- board text added: "12V"
- board text added: "3,3V"
- board text added: "BATT_IN"
- board text added: "Goaly Motherboard Designed by Pixeljoch, February 2022 Funded by Leaphy"
- board text added: "Look at my credentials"
- board text added: "MAGN"
- board text added: "MOTOR 1"
- board text added: "MOTOR 2"
- board text added: "MOTOR 3"
- board text added: "OFF"
- board text added: "OLED"
- board text added: "ON"
- board text added: "TRUST ME"
- board text added: "US_L"
- board text added: "US_R"
- board text added: "VBAT"
- board text added: "WE'RE ENGINEERS"

Commit message: Finished DRC [MAIN BOARD]
Parts:
- moved D3 1.52 mm to (93.5, 146.3)
- moved D9 1.02 mm to (205.2, 146.3)
Routing:
- net Net-(D2-Pad2): track 54.5 -> 56.1 mm
- net Net-(D3-Pad2): track 56.4 -> 54.9 mm
- net Net-(D8-Pad2): track 56.6 -> 55.5 mm

Commit message: Updated to Kicad 6
Connections:
- net ~CS renamed ~{CS}
- net ~EN renamed ~{EN}
- net ~WR renamed ~{WR}
Other:
- net class Default removed
