File: Main_Board/Main_Board.kicad_sch (KiCad schematic)
At the start: 67 parts, among them J1 Conn_01x06, J10 HR-SR04_L_CONN, J11 12V_OUT, J12 BATT_REG_IN, J13 LED_CONN, J14 PD_CONN, J2 Conn_01x06, J3 Conn_01x06, J4 BATT_IN, J5 Conn_02x08_Top_Bottom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

Commit message: Finished IR, generated gerbers, ordered designs
Parts:
- D12: value 20V -> 15V
Connections:
- net +3V3: now also J5.8 (Pin_8); no longer J5.15 (Pin_15)
- net GND: now also J5.10 (Pin_10); no longer J5.16 (Pin_16)
- net IR1: now also J5.9 (Pin_9), U1.17 (A3); no longer J5.1 (Pin_1), U1.38 (A14)
- net IR10: now also J5.14 (Pin_14), U1.24 (A10); no longer J5.10 (Pin_10), U1.19 (A5)
- net IR11: now also J5.16 (Pin_16), U1.26 (A12); no longer J5.11 (Pin_11), U1.24 (A10)
- net IR12: now also J5.15 (Pin_15), U1.27 (A13); no longer J5.12 (Pin_12), U1.25 (A11)
- net IR13: now also U1.25 (A11); no longer U1.26 (A12)
- net IR14: now also J5.11 (Pin_11), U1.19 (A5); no longer J5.14 (Pin_14), U1.27 (A13)
- net IR2: now also J5.7 (Pin_7), U1.16 (A2); no longer J5.2 (Pin_2), U1.39 (A15)
- net IR3: now also J5.5 (Pin_5), U1.14 (A0); no longer J5.3 (Pin_3), U1.40 (A16)
- net IR4: now also J5.3 (Pin_3), U1.40 (A16); no longer J5.4 (Pin_4), U1.41 (A17)
- net IR5: now also J5.1 (Pin_1), U1.38 (A14); no longer J5.5 (Pin_5), U1.14 (A0)
- net IR6: now also J5.2 (Pin_2), U1.39 (A15); no longer J5.6 (Pin_6), U1.15 (A1)
- net IR7: now also J5.4 (Pin_4), U1.41 (A17); no longer J5.7 (Pin_7), U1.16 (A2)
- net IR8: now also J5.6 (Pin_6), U1.15 (A1); no longer J5.8 (Pin_8), U1.17 (A3)
- net IR9: now also J5.12 (Pin_12); no longer J5.9 (Pin_9)
